File: mcdanibj/project-1/project-1.kicad_sch (KiCad schematic)
At the start: 7 parts, among them J1 Conn_01x04

Commit message: aaaaa
Parts:
- added H1: MountingHole, MountingHole:MountingHole_2.2mm_M2, symbol Mechanical:MountingHole
Other:
- added sheet sd-card-read (sd-card-reader.kicad_sch)
Changed lines of the file:
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@@
+    )
+  )
+  (symbol (lib_id "Mechanical:MountingHole") (at 149.86 34.29 0) (unit 1)
+    (in_bom yes) (on_board yes) (dnp no) (fields_autoplaced)
+    (property "Reference" "H1" (at 152.4 33.02 0)
+      (effects (font (size 1.27 1.27)) (justify left))
+    )
+    (property "Value" "MountingHole" (at 152.4 35.56 0)
+      (effects (font (size 1.27 1.27)) (justify left))
+    )
+    (property "Footprint" "MountingHole:MountingHole_2.2mm_M2" (at 149.86 34.29 0)
+      (effects (font (size 1.27 1.27)) hide)
+    )
+    (property "Datasheet" "~" (at 149.86 34.29 0)
+      (effects (font (size 1.27 1.27)) hide)
+    )
+    (instances
+      (project "project-1"
+        (path "/f3ab6f32-0e59-47bc-9fc0-c99654fd7e83"
+          (reference "H1") (unit 1)
+        )
+      )
     )
   )
@@
       )
     )
+  )
+  (sheet (at 86.36 78.74) (size 33.02 17.78) (fields_autoplaced)
+    (stroke (width 0.1524) (type solid))
+    (fill (color 0 0 0 0.0000))
+    (property "Sheetname" "sd-card-read" (at 86.36 78.0284 0)
+      (effects (font (size 1.27 1.27)) (justify left bottom))
+    )
+    (property "Sheetfile" "sd-card-reader.kicad_sch" (at 86.36 97.1046 0)
+      (effects (font (size 1.27 1.27)) (justify left top))
+    )
+    (pin "data_0" input (at 119.38 82.55 0)
+      (effects (font (size 1.27 1.27)) (justify right))
+    )
+    (pin "data_1" input (at 119.38 85.09 0)
+      (effects (font (size 1.27 1.27)) (justify right))
+    )
+    (instances
+      (project "project-1"
+        (path "/f3ab6f32-0e59-47bc-9fc0-c99654fd7e83" (page "2"))
+      )
+    )
