File: Ian Kirschenbaum/project 1/project 1.kicad_pcb (KiCad board)
At the start: 2 copper layers, 7 parts, among them J1 Conn_01x04

Commit message: update
Parts:
- added D4: LED, LED_THT:LED_D3.0mm, F.Cu at (139.7, 66.0)
- added H1: MountingHole, MountingHole:MountingHole_6.5mm, F.Cu at (134.6, 129.5)
- added R4: R, Resistor_THT:R_Axial_DIN0411_L9.9mm_D3.6mm_P12.70mm_Horizontal, F.Cu at (139.7, 41.9)
- J1: value Conn_01x04 -> Conn_2Rows-05Pins; footprint Connector_PinHeader_2.00mm:PinHeader_1x04_P2.00mm_Horizontal -> Connector_PinHeader_2.54mm:PinHeader_1x05_P2.54mm_Horizontal
- moved J1 112.9 mm to (86.4, 27.9), turned to 90 degrees
- moved D1 93.4 mm to (76.2, 111.8), turned to 90 degrees
- moved R1 89.6 mm to (76.2, 72.4)
- moved R3 89.0 mm to (101.6, 43.2), turned to 0 degrees
- moved R2 86.9 mm to (88.9, 59.7), turned to -90 degrees
- moved D2 86.4 mm to (88.9, 111.8), turned to 90 degrees
- moved D3 60.6 mm to (121.9, 43.2), turned to 180 degrees
Connections:
- D1 pad 1: Net-(D1-K) -> unconnected-(D1-K-Pad1)
- D2 pad 1: Net-(D1-K) -> unconnected-(D2-K-Pad1)
- D3 pad 1: Net-(D1-K) -> unconnected-(D3-K-Pad1)
- J1 pad 4: Net-(D1-K) -> Net-(J1-Pin_4)
- R1 pad 1: Net-(J1-Pin_3) -> Net-(D1-A)
- R1 pad 2: Net-(D3-A) -> Net-(J1-Pin_1)
- R3 pad 1: Net-(J1-Pin_1) -> Net-(J1-Pin_3)
- R3 pad 2: Net-(D1-A) -> Net-(D3-A)
Routing:
- net unconnected-(J1-Pin_5-Pad5): track 0.00 -> 235.8 mm
- net Net-(J1-Pin_4): track 0.00 -> 54.5 mm
- net Net-(D2-A): track 0.00 -> 36.8 mm
- net Net-(D1-A): track 0.00 -> 36.8 mm
- net Net-(J1-Pin_1): track 8.90 -> 36.0 mm
- net Net-(J1-Pin_2): track 7.65 -> 31.7 mm
- net Net-(J1-Pin_3): track 8.92 -> 23.9 mm
- net Net-(D4-A): track 0.00 -> 8.89 mm
- net Net-(D3-A): track 0.00 -> 5.08 mm
Other:
- board outline added: 109.2 x 121.9 mm
