File: Ian Kirschenbaum/project 1/project 1.kicad_sch (KiCad schematic)
At the start: 7 parts, among them J1 Conn_01x04

Commit message: update
Parts:
- removed J1: Conn_01x04, symbol Connector_Generic:Conn_01x04
- added D4: LED, LED_THT:LED_D3.0mm, symbol Device:LED
- added H1: MountingHole, MountingHole:MountingHole_6.5mm, symbol Mechanical:MountingHole
- added J1: Conn_2Rows-05Pins, Connector_PinHeader_2.54mm:PinHeader_1x05_P2.54mm_Horizontal, symbol Connector_Generic:Conn_2Rows-05Pins
- added R4: R, Resistor_THT:R_Axial_DIN0411_L9.9mm_D3.6mm_P12.70mm_Horizontal, symbol Device:R
- D1, D2, D3: footprint (none) -> LED_THT:LED_D3.0mm
- R1, R2, R3: footprint (none) -> Resistor_THT:R_Axial_DIN0411_L9.9mm_D3.6mm_P12.70mm_Horizontal
Connections:
- net at R2.1: now also J1.2 (Pin_2)
- net at D1.2 (A): now also R1.1; no longer R3.2
- net at R3.1: now also J1.3 (Pin_3)
- net at R1.2: now also J1.1 (Pin_1); no longer D3.2 (A)
- new net: J1.4 (Pin_4), R4.1
- new net: D4.2 (A), R4.2
- new net: D3.2 (A), R3.2
- now unconnected: D1.1 (K), D2.1 (K), D3.1 (K)
Other:
- moved on the sheet: D1, D2, D3, R1, R2, R3
