File: noname-board/power/power.kicad_sch (KiCad schematic)
At the start: 9 parts, among them J1 Conn_01x02_Pin, Q1 LM2940CT-5.0_NOPB

Commit message: fixed ben's whoopsie
Parts:
- removed C1: .47uF, Capacitor_THT:CP_Radial_D5.0mm_P2.00mm, symbol Device:C
- removed C2: 22uF, Capacitor_THT:CP_Radial_D5.0mm_P2.00mm, symbol Device:C
- removed C3: 10uF, symbol Device:C
- removed C4: 10uF MUST BE TANTALUM, symbol Device:C
- removed J1: Conn_01x02_Pin, XT30:XT30UPB-M, symbol Connector:Conn_01x02_Pin
- removed PS2: LM1084IT-3.3_NOPB, TO254P470X1028X1955-3P, symbol LM1084IT-3.3NOPB:LM1084IT-3.3_NOPB
- removed Q1: LM2940CT-5.0_NOPB, TO254P470X1028X1955-3P, symbol LM2940CT-5.0/NOPB:LM2940CT-5.0_NOPB
- removed R1: 121 Nominal, symbol Device:R
- removed R2: 5k, symbol Device:R_Variable_US
Other:
- added sheet POWER (power_hehe.kicad_sch)
