File: noname-board/power/power_hehe.kicad_sch (KiCad schematic)
At the start: 9 parts, among them J1 Conn_01x02_Pin, Q1 LM2940CT-5.0_NOPB

Commit message: We went thru eveeeryyything
Connections:
- net GND is gone; now on net GND_xt30: Q1.2 (GND)
Changed lines of the file:
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@@
   (junction (at 93.98 78.74) (diameter 0) (color 0 0 0 0)
+  )
+  (junction (at 113.03 120.65) (diameter 0) (color 0 0 0 0)
   )
   (junction (at 93.98 120.65) (diameter 0) (color 0 0 0 0)
@@
     (stroke (width 0) (type default))
   )
+  (wire (pts (xy 113.03 120.65) (xy 125.73 120.65))
+    (stroke (width 0) (type default))
+  )
   (wire (pts (xy 144.78 68.58) (xy 144.78 78.74))
     (stroke (width 0) (type default))
@@
     (stroke (width 0) (type default))
   )
-  (wire (pts (xy 113.03 110.49) (xy 113.03 109.22))
+  (wire (pts (xy 113.03 109.22) (xy 113.03 120.65))
     (stroke (width 0) (type default))
   )
@@
     (stroke (width 0) (type default))
   )
-  (wire (pts (xy 100.33 120.65) (xy 125.73 120.65))
+  (wire (pts (xy 100.33 120.65) (xy 113.03 120.65))
     (stroke (width 0) (type default))
   )
@@
     (stroke (width 0) (type default))
   )
-  (global_label "GND" (shape input) (at 113.03 110.49 270) (fields_autoplaced)
-    (effects (font (size 1.27 1.27)) (justify right))
-    (property "Intersheetrefs" "${INTERSHEET_REFS}" (at 113.03 117.3457 90)
-      (effects (font (size 1.27 1.27)) (justify right) hide)
-    )
-  )
   (hierarchical_label "5V" (shape input) (at 139.7 110.49 0) (fields_autoplaced)
