File: eieminia_Luci/Project_1/Project_1.kicad_sch (KiCad schematic)
At the start: 7 parts, among them J1 Conn_01x04

Commit message: USBC Thingy
Parts:
- removed J1: Conn_01x04, Connector_PinHeader_2.00mm:PinHeader_1x04_P2.00mm_Horizontal, symbol Connector_Generic:Conn_01x04
- added D4: LED, LED_THT:LED_D3.0mm, symbol Device:LED
- added H1: MountingHole, MountingHole:MountingHole_2.2mm_M2, symbol Mechanical:MountingHole
- added J2: Conn_01x05, Connector_PinHeader_2.54mm:PinHeader_1x05_P2.54mm_Horizontal, symbol Connector_Generic:Conn_01x05
- added R4: R, Resistor_THT:R_Axial_DIN0411_L9.9mm_D3.6mm_P12.70mm_Horizontal, symbol Device:R
Connections:
- net at R1.1: now also J2.4 (Pin_4)
- net at D1.1 (K), D2.1 (K), D3.1 (K): now also D4.1 (K), J2.5 (Pin_5)
- net at R2.1: now also J2.3 (Pin_3)
- net at R3.1: now also J2.2 (Pin_2)
- new net: D4.2 (A), R4.2
- new net: J2.1 (Pin_1), R4.1
Changed lines of the file:
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@@
 (kicad_sch (version 20230121) (generator eeschema)
   (paper "A4")
+  (junction (at 80.01 76.2) (diameter 0) (color 0 0 0 0)
+  )
   (junction (at 80.01 63.5) (diameter 0) (color 0 0 0 0)
   )
   (junction (at 80.01 50.8) (diameter 0) (color 0 0 0 0)
   )
-  (wire (pts (xy 31.75 39.37) (xy 80.01 39.37))
-    (stroke (width 0) (type default))
-  )
-  (wire (pts (xy 31.75 68.58) (xy 49.53 68.58))
-    (stroke (width 0) (type default))
-  )
-  (wire (pts (xy 43.18 66.04) (xy 43.18 50.8))
+  (wire (pts (xy 30.48 39.37) (xy 80.01 39.37))
+    (stroke (width 0) (type default))
+  )
+  (wire (pts (xy 33.02 67.31) (xy 33.02 63.5))
+    (stroke (width 0) (type default))
+  )
+  (wire (pts (xy 71.12 85.09) (xy 80.01 85.09))
     (stroke (width 0) (type default))
   )
@@
     (stroke (width 0) (type default))
   )
-  (wire (pts (xy 49.53 68.58) (xy 49.53 63.5))
-    (stroke (width 0) (type default))
-  )
-  (wire (pts (xy 31.75 66.04) (xy 43.18 66.04))
-    (stroke (width 0) (type default))
-  )
-  (wire (pts (xy 49.53 71.12) (xy 49.53 76.2))
+  (wire (pts (xy 30.48 69.85) (xy 49.53 69.85))
+    (stroke (width 0) (type default))
+  )
+  (wire (pts (xy 49.53 69.85) (xy 49.53 76.2))
+    (stroke (width 0) (type default))
+  )
+  (wire (pts (xy 30.48 67.31) (xy 33.02 67.31))
+    (stroke (width 0) (type default))
+  )
+  (wire (pts (xy 46.99 85.09) (xy 49.53 85.09))
     (stroke (width 0) (type default))
   )
@@
     (stroke (width 0) (type default))
   )
+  (wire (pts (xy 33.02 63.5) (xy 49.53 63.5))
+    (stroke (width 0) (type default))
+  )
+  (wire (pts (xy 80.01 85.09) (xy 80.01 76.2))
+    (stroke (width 0) (type default))
+  )
+  (wire (pts (xy 57.15 85.09) (xy 63.5 85.09))
+    (stroke (width 0) (type default))
+  )
   (wire (pts (xy 80.01 63.5) (xy 80.01 76.2))
     (stroke (width 0) (type default))
@@
     (stroke (width 0) (type default))
   )
+  (wire (pts (xy 30.48 62.23) (xy 30.48 39.37))
+    (stroke (width 0) (type default))
+  )
+  (wire (pts (xy 31.75 64.77) (xy 31.75 50.8))
+    (stroke (width 0) (type default))
+  )
   (wire (pts (xy 57.15 50.8) (xy 63.5 50.8))
     (stroke (width 0) (type default))
   )
+  (wire (pts (xy 30.48 72.39) (xy 46.99 72.39))
+    (stroke (width 0) (type default))
+  )
   (wire (pts (xy 57.15 76.2) (xy 63.5 76.2))
     (stroke (width 0) (type default))
   )
-  (wire (pts (xy 31.75 71.12) (xy 49.53 71.12))
+  (wire (pts (xy 30.48 64.77) (xy 31.75 64.77))
     (stroke (width 0) (type default))
   )
@@
     (stroke (width 0) (type default))
   )
+  (wire (pts (xy 46.99 72.39) (xy 46.99 85.09))
+    (stroke (width 0) (type default))
+  )
   (wire (pts (xy 80.01 39.37) (xy 80.01 50.8))
     (stroke (width 0) (type default))
@@
     (stroke (width 0) (type default))
   )
-  (wire (pts (xy 31.75 63.5) (xy 31.75 39.37))
-    (stroke (width 0) (type default))
-  )
-  (wire (pts (xy 43.18 50.8) (xy 49.53 50.8))
+  (wire (pts (xy 31.75 50.8) (xy 49.53 50.8))
     (stroke (width 0) (type default))
   )
@@
     )
   )
+  (symbol (lib_id "Mechanical:MountingHole") (at 40.64 45.72 0) (unit 1)
+    (in_bom yes) (on_board yes) (dnp no) (fields_autoplaced)
+    (property "Reference" "H1" (at 43.18 44.45 0)
+      (effects (font (size 1.27 1.27)) (justify left))
+    )
+    (property "Value" "MountingHole" (at 43.18 46.99 0)
+      (effects (font (size 1.27 1.27)) (justify left))
+    )
+    (property "Footprint" "MountingHole:MountingHole_2.2mm_M2" (at 40.64 45.72 0)
+      (effects (font (size 1.27 1.27)) hide)
+    )
+    (property "Datasheet" "~" (at 40.64 45.72 0)
+      (effects (font (size 1.27 1.27)) hide)
+    )
+    (instances
+      (project "Project_1"
+        (path "/8ec92794-c088-4c63-b3f8-cd21d727fc94"
+          (reference "H1") (unit 1)
+        )
+      )
+    )
+  )
   (symbol (lib_id "Device:LED") (at 67.31 76.2 180) (unit 1)
     (in_bom yes) (on_board yes) (dnp no) (fields_autoplaced)
@@
     )
   )
-  (symbol (lib_id "Device:LED") (at 67.31 63.5 180) (unit 1)
-    (in_bom yes) (on_board yes) (dnp no) (fields_autoplaced)
-    (property "Reference" "D2" (at 68.8975 55.88 0)
-      (effects (font (size 1.27 1.27)))
-    )
-    (property "Value" "LED" (at 68.8975 58.42 0)
-      (effects (font (size 1.27 1.27)))
-    )
-    (property "Footprint" "LED_THT:LED_D3.0mm" (at 67.31 63.5 0)
-      (effects (font (size 1.27 1.27)) hide)
-    )
-    (property "Datasheet" "~" (at 67.31 63.5 0)
-      (effects (font (size 1.27 1.27)) hide)
-    )
-    (pin "1")
-    (pin "2")
-    (instances
-      (project "Project_1"
-        (path "/8ec92794-c088-4c63-b3f8-cd21d727fc94"
-          (reference "D2") (unit 1)
-        )
-      )
-    )
-  )
-  (symbol (lib_id "Connector_Generic:Conn_01x04") (at 26.67 68.58 180) (unit 1)
-    (in_bom yes) (on_board yes) (dnp no) (fields_autoplaced)
-    (property "Reference" "J1" (at 26.67 57.15 0)
-      (effects (font (size 1.27 1.27)))
-    )
-    (property "Value" "Conn_01x04" (at 26.67 59.69 0)
-      (effects (font (size 1.27 1.27)))
-    )
-    (property "Footprint" "Connector_PinHeader_2.00mm:PinHeader_1x04_P2.00mm_Horizontal" (at 26.67 68.58 0)
-      (effects (font (size 1.27 1.27)) hide)
-    )
-    (property "Datasheet" "~" (at 26.67 68.58 0)
+  (symbol (lib_id "Device:LED") (at 67.31 85.09 180) (unit 1)
+    (in_bom yes) (on_board yes) (dnp no) (fields_autoplaced)
+    (property "Reference" "D4" (at 68.8975 77.47 0)
+      (effects (font (size 1.27 1.27)))
+    )
+    (property "Value" "LED" (at 68.8975 80.01 0)
+      (effects (font (size 1.27 1.27)))
+    )
+    (property "Footprint" "LED_THT:LED_D3.0mm" (at 67.31 85.09 0)
+      (effects (font (size 1.27 1.27)) hide)
+    )
+    (property "Datasheet" "~" (at 67.31 85.09 0)
+      (effects (font (size 1.27 1.27)) hide)
+    )
+    (pin "1")
+    (pin "2")
+    (instances
+      (project "Project_1"
+        (path "/8ec92794-c088-4c63-b3f8-cd21d727fc94"
+          (reference "D4") (unit 1)
+        )
+      )
+    )
+  )
+  (symbol (lib_id "Connector_Generic:Conn_01x05") (at 25.4 67.31 180) (unit 1)
+    (in_bom yes) (on_board yes) (dnp no) (fields_autoplaced)
+    (property "Reference" "J2" (at 25.4 55.88 0)
+      (effects (font (size 1.27 1.27)))
+    )
+    (property "Value" "Conn_01x05" (at 25.4 58.42 0)
+      (effects (font (size 1.27 1.27)))
+    )
+    (property "Footprint" "Connector_PinHeader_2.54mm:PinHeader_1x05_P2.54mm_Horizontal" (at 25.4 67.31 0)
+      (effects (font (size 1.27 1.27)) hide)
+    )
+    (property "Datasheet" "~" (at 25.4 67.31 0)
       (effects (font (size 1.27 1.27)) hide)
     )
@@
     (pin "3")
     (pin "4")
-    (instances
-      (project "Project_1"
-        (path "/8ec92794-c088-4c63-b3f8-cd21d727fc94"
-          (reference "J1") (unit 1)
+    (pin "5")
+    (instances
+      (project "Project_1"
+        (path "/8ec92794-c088-4c63-b3f8-cd21d727fc94"
+          (reference "J2") (unit 1)
+        )
+      )
+    )
+  )
+  (symbol (lib_id "Device:LED") (at 67.31 63.5 180) (unit 1)
+    (in_bom yes) (on_board yes) (dnp no) (fields_autoplaced)
+    (property "Reference" "D2" (at 68.8975 55.88 0)
+      (effects (font (size 1.27 1.27)))
+    )
+    (property "Value" "LED" (at 68.8975 58.42 0)
+      (effects (font (size 1.27 1.27)))
+    )
+    (property "Footprint" "LED_THT:LED_D3.0mm" (at 67.31 63.5 0)
+      (effects (font (size 1.27 1.27)) hide)
+    )
+    (property "Datasheet" "~" (at 67.31 63.5 0)
+      (effects (font (size 1.27 1.27)) hide)
+    )
+    (pin "1")
+    (pin "2")
+    (instances
+      (project "Project_1"
+        (path "/8ec92794-c088-4c63-b3f8-cd21d727fc94"
+          (reference "D2") (unit 1)
         )
       )
@@
         )
       )
+    )
+  )
+  (symbol (lib_id "Device:R") (at 53.34 85.09 90) (unit 1)
+    (in_bom yes) (on_board yes) (dnp no) (fields_autoplaced)
+    (property "Reference" "R4" (at 53.34 78.74 90)
+      (effects (font (size 1.27 1.27)))
+    )
+    (property "Value" "R" (at 53.34 81.28 90)
+      (effects (font (size 1.27 1.27)))
+    )
+    (property "Footprint" "Resistor_THT:R_Axial_DIN0411_L9.9mm_D3.6mm_P12.70mm_Horizontal" (at 53.34 86.868 90)
+      (effects (font (size 1.27 1.27)) hide)
+    )
+    (property "Datasheet" "~" (at 53.34 85.09 0)
+      (effects (font (size 1.27 1.27)) hide)
+    )
+    (pin "1")
+    (pin "2")
+    (instances
+      (project "Project_1"
+        (path "/8ec92794-c088-4c63-b3f8-cd21d727fc94"
+          (reference "R4") (unit 1)
+        )
+      )

Commit message: Did Stuff
Parts:
- removed D1, D2, D3, D4: LED, LED_THT:LED_D3.0mm, symbol Device:LED
- removed H1: MountingHole, MountingHole:MountingHole_2.2mm_M2, symbol Mechanical:MountingHole
- removed J2: Conn_01x05, Connector_PinHeader_2.54mm:PinHeader_1x05_P2.54mm_Horizontal, symbol Connector_Generic:Conn_01x05
- removed R1, R2, R3, R4: R, Resistor_THT:R_Axial_DIN0411_L9.9mm_D3.6mm_P12.70mm_Horizontal, symbol Device:R
- added D5, D6, D7, D8: LED, LED_THT:LED_D3.0mm, symbol Device:LED
- added H2: MountingHole, MountingHole:MountingHole_2.1mm, symbol Mechanical:MountingHole
- added J1: Conn_01x05, Connector_PinHeader_2.54mm:PinHeader_1x05_P2.54mm_Horizontal, symbol Connector_Generic:Conn_01x05
- added R5, R6, R7, R8: R, Resistor_THT:R_Axial_DIN0309_L9.0mm_D3.2mm_P12.70mm_Horizontal, symbol Device:R
Connections:
- new net: D5.1 (K), D6.1 (K), D7.1 (K), D8.1 (K), J1.5 (Pin_5)
- new net: D8.2 (A), R8.2
- new net: J1.4 (Pin_4), R5.1
- new net: D5.2 (A), R5.2
- new net: J1.3 (Pin_3), R6.1
- new net: D6.2 (A), R6.2
- new net: D7.2 (A), R7.2
- new net: J1.2 (Pin_2), R7.1
- new net: J1.1 (Pin_1), R8.1
