File: noname-board/ROSE-PILK_v1/_autosave-ROSE-PILK_v1.kicad_sch (KiCad schematic)
At the start: 2 parts, among them J2 Conn_01x03, SW1 SW_Push

Commit message: Team Meeting
Dear Diary,
today i had a thing
it was a horrible thing
a very horrible horrible thing
i hated it
Changed lines of the file:
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@@
     (stroke (width 0) (type default))
   )
-  (wire (pts (xy 78.74 67.31) (xy 78.74 71.12))
+  (wire (pts (xy 80.01 67.31) (xy 80.01 71.12))
     (stroke (width 0) (type default))
   )
@@
     (stroke (width 0) (type default))
   )
-  (wire (pts (xy 81.28 67.31) (xy 78.74 67.31))
+  (wire (pts (xy 81.28 67.31) (xy 80.01 67.31))
     (stroke (width 0) (type default))
   )
@@
     (stroke (width 0) (type default))
   )
-  (wire (pts (xy 78.74 71.12) (xy 74.93 71.12))
+  (wire (pts (xy 80.01 71.12) (xy 74.93 71.12))
     (stroke (width 0) (type default))
   )
