File: noname-board/ROSE-PILK_v1/_autosave-ROSE-PILK_v1.kicad_pcb (KiCad board)
At the start: 2 copper layers, 83 parts, among them J1 USB_C_Receptacle, J2 Conn_01x03, J3 Conn_01x02, J4 Conn_01x02, J5 Conn_02x08_Row_Letter_First, J6 Conn_01x03, J6 Conn_01x03_Pin, J7 Conn_02x08_Row_Letter_Last, Q3 PN2222A, SW1 SW_Push, SW3 SW_Push_Dual, U1 W25Q128JVS, U2 ASDMB-12MHz, U3 RP2040

Commit message: BootSel
Parts:
- added PS1: LM1084IT-3.3_NOPB, LM1084IT-3.3:TO254P1054X470X1955-3, F.Cu at (154.9, 109.1)
- added Q1: LM2940CT-5.0_NOPB, LM2940CT-5.0:TO254P1054X470X1955-3, F.Cu at (154.9, 116.0)
- added U4: XT30UPB-M, XT30UPB-M:XT30UPB-M, F.Cu at (154.5, 122.4)
- added U5: SN65HVD230DR, SN65HVD230DR:SOIC127P599X175-8N, F.Cu at (167.7, 127.6)
- added U6: CD4514BM, CD4514BM:SOIC127P1030X265-24N, F.Cu at (170.4, 113.9)
- added U7: SN65HVD230DR, SN65HVD230DR:SOIC127P599X175-8N, F.Cu at (153.6, 130.8)
- SW3: footprint Button_Switch_THT:SW_PUSH_6mm -> Button_Switch_THT:SW_CuK_JS202011CQN_DPDT_Straight
