File: noname-board/ROSE-PILK_v1/CAN2.kicad_sch (KiCad schematic)
At the start: 3 parts, among them J3 Conn_01x02, U5 SN65HVD230DR

Commit message: Meeting Stuff
Parts:
- removed J3: Conn_01x02, ul_SM02B-GHS-TB:CONN_SM02B-GHS-TB_JST, symbol Connector_Generic:Conn_01x02
- added J4: Conn_01x04, SM04B_GHS_TB_LF__SN__:JST_SM04B-GHS-TB_LF__SN_-, symbol Connector_Generic:Conn_01x04
Connections:
- net GND: now also J4.3 (Pin_3)
- net at R32.2, U5.6 (CANL): now also J4.1 (Pin_1)
- net at R32.1, U5.7 (CANH): now also J4.2 (Pin_2)
- new net 5V: J4.4 (Pin_4)
Changed lines of the file:
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@@
 (kicad_sch (version 20230121) (generator eeschema)
   (paper "A4")
-  (junction (at 191.77 54.61) (diameter 0) (color 0 0 0 0)
+  (junction (at 179.07 90.17) (diameter 0) (color 0 0 0 0)
   )
-  (junction (at 191.77 62.23) (diameter 0) (color 0 0 0 0)
+  (junction (at 179.07 82.55) (diameter 0) (color 0 0 0 0)
   )
-  (no_connect (at 172.72 62.23))
-  (wire (pts (xy 110.49 62.23) (xy 116.84 62.23))
+  (no_connect (at 160.02 90.17))
+  (wire (pts (xy 160.02 74.93) (xy 160.02 82.55))
     (stroke (width 0) (type default))
   )
-  (wire (pts (xy 172.72 46.99) (xy 172.72 54.61))
+  (wire (pts (xy 179.07 82.55) (xy 190.5 82.55))
     (stroke (width 0) (type default))
   )
-  (wire (pts (xy 110.49 57.15) (xy 116.84 57.15))
+  (wire (pts (xy 165.1 85.09) (xy 165.1 82.55))
     (stroke (width 0) (type default))
   )
-  (wire (pts (xy 191.77 62.23) (xy 177.8 62.23))
+  (wire (pts (xy 97.79 90.17) (xy 104.14 90.17))
     (stroke (width 0) (type default))
   )
-  (wire (pts (xy 191.77 54.61) (xy 210.82 54.61))
+  (wire (pts (xy 201.93 87.63) (xy 190.5 87.63))
     (stroke (width 0) (type default))
   )
-  (wire (pts (xy 177.8 54.61) (xy 191.77 54.61))
+  (wire (pts (xy 165.1 90.17) (xy 165.1 87.63))
     (stroke (width 0) (type default))
   )
-  (wire (pts (xy 199.39 57.15) (xy 199.39 62.23))
+  (wire (pts (xy 165.1 82.55) (xy 179.07 82.55))
     (stroke (width 0) (type default))
   )
-  (wire (pts (xy 199.39 62.23) (xy 191.77 62.23))
+  (wire (pts (xy 190.5 82.55) (xy 190.5 87.63))
     (stroke (width 0) (type default))
   )
-  (wire (pts (xy 172.72 59.69) (xy 177.8 59.69))
+  (wire (pts (xy 97.79 85.09) (xy 104.14 85.09))
     (stroke (width 0) (type default))
   )
-  (wire (pts (xy 177.8 62.23) (xy 177.8 59.69))
+  (wire (pts (xy 179.07 90.17) (xy 165.1 90.17))
     (stroke (width 0) (type default))
   )
-  (wire (pts (xy 199.39 57.15) (xy 210.82 57.15))
+  (wire (pts (xy 179.07 90.17) (xy 201.93 90.17))
     (stroke (width 0) (type default))
   )
-  (wire (pts (xy 110.49 54.61) (xy 116.84 54.61))
+  (wire (pts (xy 97.79 82.55) (xy 104.14 82.55))
     (stroke (width 0) (type default))
   )
-  (wire (pts (xy 177.8 57.15) (xy 177.8 54.61))
+  (wire (pts (xy 97.79 87.63) (xy 104.14 87.63))
     (stroke (width 0) (type default))
   )
-  (wire (pts (xy 110.49 59.69) (xy 116.84 59.69))
+  (wire (pts (xy 160.02 85.09) (xy 165.1 85.09))
     (stroke (width 0) (type default))
   )
-  (wire (pts (xy 172.72 57.15) (xy 177.8 57.15))
+  (wire (pts (xy 160.02 87.63) (xy 165.1 87.63))
     (stroke (width 0) (type default))
   )
-  (text "CAN_L" (at 204.47 59.69 0)
+  (text "CAN_H\n" (at 190.5 87.63 0)
     (effects (font (size 1.27 1.27)) (justify left bottom))
   )
-  (text "CAN_H\n" (at 204.47 54.61 0)
+  (text "CAN_L" (at 190.5 92.71 0)
     (effects (font (size 1.27 1.27)) (justify left bottom))
   )
-  (hierarchical_label "GND" (shape input) (at 172.72 46.99 90) (fields_autoplaced)
+  (hierarchical_label "GND" (shape input) (at 97.79 85.09 180) (fields_autoplaced)
+    (effects (font (size 1.27 1.27)) (justify right))
+  )
+  (hierarchical_label "GND" (shape input) (at 160.02 74.93 90) (fields_autoplaced)
     (effects (font (size 1.27 1.27)) (justify left))
   )
-  (hierarchical_label "CAN_TX" (shape input) (at 110.49 54.61 180) (fields_autoplaced)
+  (hierarchical_label "5V" (shape input) (at 201.93 82.55 180) (fields_autoplaced)
     (effects (font (size 1.27 1.27)) (justify right))
   )
-  (hierarchical_label "3V3" (shape input) (at 110.49 59.69 180) (fields_autoplaced)
+  (hierarchical_label "CAN_TX" (shape input) (at 97.79 82.55 180) (fields_autoplaced)
     (effects (font (size 1.27 1.27)) (justify right))
   )
-  (hierarchical_label "CAN_RX" (shape input) (at 110.49 62.23 180) (fields_autoplaced)
+  (hierarchical_label "CAN_RX" (shape input) (at 97.79 90.17 180) (fields_autoplaced)
     (effects (font (size 1.27 1.27)) (justify right))
   )
-  (hierarchical_label "GND" (shape input) (at 110.49 57.15 180) (fields_autoplaced)
+  (hierarchical_label "3V3" (shape input) (at 97.79 87.63 180) (fields_autoplaced)
     (effects (font (size 1.27 1.27)) (justify right))
   )
-  (symbol (lib_id "SN65HVD230DR:SN65HVD230DR") (at 116.84 54.61 0) (unit 1)
+  (hierarchical_label "GND" (shape input) (at 201.93 85.09 180) (fields_autoplaced)
+    (effects (font (size 1.27 1.27)) (justify right))
+  )
+  (symbol (lib_id "SN65HVD230DR:SN65HVD230DR") (at 104.14 82.55 0) (unit 1)
     (in_bom yes) (on_board yes) (dnp no) (fields_autoplaced)
-    (property "Reference" "U5" (at 144.78 44.45 0)
+    (property "Reference" "U5" (at 132.08 72.39 0)
       (effects (font (size 1.524 1.524)))
     )
-    (property "Value" "SN65HVD230DR" (at 144.78 46.99 0)
+    (property "Value" "SN65HVD230DR" (at 132.08 74.93 0)
       (effects (font (size 1.524 1.524)))
     )
-    (property "Footprint" "SN65HVD230DR:SOIC127P599X175-8N" (at 116.84 54.61 0)
+    (property "Footprint" "SN65HVD230DR:SOIC127P599X175-8N" (at 104.14 82.55 0)
       (effects (font (size 1.27 1.27) italic) hide)
     )
-    (property "Datasheet" "SN65HVD230DR" (at 116.84 54.61 0)
+    (property "Datasheet" "SN65HVD230DR" (at 104.14 82.55 0)
       (effects (font (size 1.27 1.27) italic) hide)
     )
@@
           (reference "U5") (unit 1)
         )
+        (path "/3dfb9737-68ba-4ca9-8085-72e4f57f9e50/cc566290-d472-48a8-a9ae-4e54f87660da"
+          (reference "U7") (unit 1)
+        )
       )
     )
   )
-  (symbol (lib_id "Connector_Generic:Conn_01x02") (at 215.9 54.61 0) (unit 1)
-    (in_bom yes) (on_board yes) (dnp no) (fields_autoplaced)
-    (property "Reference" "J3" (at 218.44 54.61 0)
+  (symbol (lib_id "Connector_Generic:Conn_01x04") (at 207.01 87.63 0) (mirror x) (unit 1)
+    (in_bom yes) (on_board yes) (dnp no)
+    (property "Reference" "J4" (at 209.55 87.63 0)
       (effects (font (size 1.27 1.27)) (justify left))
     )
-    (property "Value" "Conn_01x02" (at 218.44 57.15 0)
+    (property "Value" "Conn_01x04" (at 209.55 85.09 0)
       (effects (font (size 1.27 1.27)) (justify left))
     )
-    (property "Footprint" "ul_SM02B-GHS-TB:CONN_SM02B-GHS-TB_JST" (at 215.9 54.61 0)
+    (property "Footprint" "SM04B_GHS_TB_LF__SN__:JST_SM04B-GHS-TB_LF__SN_-" (at 207.01 87.63 0)
       (effects (font (size 1.27 1.27)) hide)
     )
-    (property "Datasheet" "~" (at 215.9 54.61 0)
+    (property "Datasheet" "~" (at 207.01 87.63 0)
       (effects (font (size 1.27 1.27)) hide)
     )
     (pin "1")
     (pin "2")
+    (pin "3")
+    (pin "4")
     (instances
       (project "ROSE-PILK_v1"
-        (path "/3dfb9737-68ba-4ca9-8085-72e4f57f9e50/abb9055d-d7a5-4a66-9ad8-cbb9f9c14958"
-          (reference "J3") (unit 1)
+        (path "/3dfb9737-68ba-4ca9-8085-72e4f57f9e50/cc566290-d472-48a8-a9ae-4e54f87660da"
+          (reference "J4") (unit 1)
         )
       )
     )
   )
-  (symbol (lib_id "Device:R") (at 191.77 58.42 0) (unit 1)
+  (symbol (lib_id "Device:R") (at 179.07 86.36 0) (unit 1)
     (in_bom yes) (on_board yes) (dnp no) (fields_autoplaced)
-    (property "Reference" "R32" (at 194.31 57.15 0)
+    (property "Reference" "R32" (at 181.61 85.09 0)
       (effects (font (size 1.27 1.27)) (justify left))
     )
-    (property "Value" "120" (at 194.31 59.69 0)
+    (property "Value" "120" (at 181.61 87.63 0)
       (effects (font (size 1.27 1.27)) (justify left))
     )
-    (property "Footprint" "Resistor_THT:R_Axial_DIN0207_L6.3mm_D2.5mm_P10.16mm_Horizontal" (at 189.992 58.42 90)
+    (property "Footprint" "Resistor_THT:R_Axial_DIN0207_L6.3mm_D2.5mm_P10.16mm_Horizontal" (at 177.292 86.36 90)
       (effects (font (size 1.27 1.27)) hide)
     )
-    (property "Datasheet" "~" (at 191.77 58.42 0)
+    (property "Datasheet" "~" (at 179.07 86.36 0)
       (effects (font (size 1.27 1.27)) hide)
     )
@@
           (reference "R32") (unit 1)
         )
+        (path "/3dfb9737-68ba-4ca9-8085-72e4f57f9e50/cc566290-d472-48a8-a9ae-4e54f87660da"
+          (reference "R33") (unit 1)
+        )
       )
