File: noname-board/ROSE-PILK_v1/DR16.kicad_sch (KiCad schematic)
At the start: 4 parts, among them J2 Conn_01x03, Q3 PN2222A

Commit message: Schematics
Parts:
- J2: footprint Connector_PinHeader_2.00mm:PinHeader_1x03_P2.00mm_Horizontal -> Connector_PinHeader_2.00mm:PinHeader_1x03_P2.00mm_Vertical
Changed lines of the file:
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@@
       (effects (font (size 1.27 1.27)))
     )
-    (property "Footprint" "Connector_PinHeader_2.00mm:PinHeader_1x03_P2.00mm_Horizontal" (at 138.43 95.25 0)
+    (property "Footprint" "Connector_PinHeader_2.00mm:PinHeader_1x03_P2.00mm_Vertical" (at 138.43 95.25 0)
       (effects (font (size 1.27 1.27)) hide)
     )
