File: noname-board/ROSE-PILK_v1/USBC.kicad_sch (KiCad schematic)
At the start: 3 parts, among them J1 USB_C_Receptacle

Commit message: dual rp2040z
Parts:
- added SW3: SW_Push_DPDT, symbol Switch:SW_Push_DPDT
Connections:
- net USB_D+ renamed D+
- net D+: now also SW3.2 (B)
- net USB_D- renamed D-
- net D-: now also SW3.5 (B)
- new net A-USB_D+: SW3.1 (A)
- new net A-USB_D-: SW3.4 (A)
- new net B-USB_D+: SW3.3 (C)
- new net B-USB_D-: SW3.6 (C)
Other:
- moved on the sheet: J1, R28, R29

Commit message: Schematics
Parts:
- SW3: footprint (none) -> Button_Switch_THT:SW_CuK_JS202011CQN_DPDT_Straight
Changed lines of the file:
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@@
       (effects (font (size 1.27 1.27)))
     )
-    (property "Footprint" "" (at 181.61 68.58 0)
+    (property "Footprint" "Button_Switch_THT:SW_CuK_JS202011CQN_DPDT_Straight" (at 181.61 68.58 0)
       (effects (font (size 1.27 1.27)) hide)
     )

Commit message: v1 functionality finished
Connections:
- net USB_5V: now reaches J1.A4 (VBUS), J1.A9 (VBUS), J1.B4 (VBUS), J1.B9 (VBUS)
Changed lines of the file:
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@@
+    (stroke (width 0) (type default))
+  )
+  (wire (pts (xy 113.03 48.26) (xy 118.11 48.26))
     (stroke (width 0) (type default))
   )
@@
     (effects (font (size 1.27 1.27)) (justify left bottom))
   )
+  (hierarchical_label "USB_5V" (shape input) (at 118.11 48.26 0) (fields_autoplaced)
+    (effects (font (size 1.27 1.27)) (justify left))
+  )
   (hierarchical_label "GND" (shape input) (at 125.73 86.36 270) (fields_autoplaced)
