File: noname-board/ROSE-PILK_v1/Power_Connectors.kicad_sch (KiCad schematic)
At the start: 3 parts, among them J13 Conn_02x08_Counter_Clockwise, J14 Conn_02x08_Counter_Clockwise, J15 Conn_02x08_Counter_Clockwise

Commit message: first pass placement doone
Parts:
- added J12, J18, J19: Conn_02x08_Counter_Clockwise, Connector_PinSocket_2.00mm:PinSocket_2x08_P2.00mm_Vertical, symbol Connector_Generic:Conn_02x08_Counter_Clockwise
Connections:
- net 3V3: now also J18.1 (Pin_1), J18.10 (Pin_10), J18.11 (Pin_11), J18.12 (Pin_12), J18.13 (Pin_13), J18.14 (Pin_14), J18.15 (Pin_15), J18.16 (Pin_16), J18.2 (Pin_2), J18.3 (Pin_3), J18.4 (Pin_4), J18.5 (Pin_5), J18.6 (Pin_6), J18.7 (Pin_7), J18.8 (Pin_8), J18.9 (Pin_9)
- net 5V: now also J12.1 (Pin_1), J12.10 (Pin_10), J12.11 (Pin_11), J12.12 (Pin_12), J12.13 (Pin_13), J12.14 (Pin_14), J12.15 (Pin_15), J12.16 (Pin_16), J12.2 (Pin_2), J12.3 (Pin_3), J12.4 (Pin_4), J12.5 (Pin_5), J12.6 (Pin_6), J12.7 (Pin_7), J12.8 (Pin_8), J12.9 (Pin_9)
- net GND: now also J19.1 (Pin_1), J19.10 (Pin_10), J19.11 (Pin_11), J19.12 (Pin_12), J19.13 (Pin_13), J19.14 (Pin_14), J19.15 (Pin_15), J19.16 (Pin_16), J19.2 (Pin_2), J19.3 (Pin_3), J19.4 (Pin_4), J19.5 (Pin_5), J19.6 (Pin_6), J19.7 (Pin_7), J19.8 (Pin_8), J19.9 (Pin_9)
