File: noname-board/ROSE-PILK_v1.5/LED_array.kicad_sch (KiCad schematic)
At the start: 1 part, among them U12 CD4515BE

Commit message: Big changes
Changed lines of the file:
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@@
+    (stroke (width 0) (type default))
+  )
+  (wire (pts (xy 173.99 111.76) (xy 180.34 111.76))
     (stroke (width 0) (type default))
   )
@@
     (effects (font (size 1.27 1.27)) (justify right))
   )
-  (hierarchical_label "GND" (shape input) (at 180.34 111.76 180) (fields_autoplaced)
+  (hierarchical_label "GND" (shape input) (at 173.99 111.76 180) (fields_autoplaced)
     (effects (font (size 1.27 1.27)) (justify right))
   )
