File: noname-board/ROSE-PILK_v1.5/LEDx15.kicad_sch (KiCad schematic)
At the start: 30 parts

Commit message: Big changes
Parts:
- added D18: WP154A4SUREQBFZGC, WP154A4SUREQBFZGC:LED_WP154A4SUREQBFZGC, symbol WP154A4SUREQBFZGC:WP154A4SUREQBFZGC
Changed lines of the file:
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@@
+    )
+  )
+  (symbol (lib_id "WP154A4SUREQBFZGC:WP154A4SUREQBFZGC") (at 97.79 129.54 0) (unit 1)
+    (in_bom yes) (on_board yes) (dnp no) (fields_autoplaced)
+    (property "Reference" "D18" (at 96.67 113.03 0)
+      (effects (font (size 1.27 1.27)))
+    )
+    (property "Value" "WP154A4SUREQBFZGC" (at 96.67 115.57 0)
+      (effects (font (size 1.27 1.27)))
+    )
+    (property "Footprint" "WP154A4SUREQBFZGC:LED_WP154A4SUREQBFZGC" (at 97.79 129.54 0)
+      (effects (font (size 1.27 1.27)) (justify bottom) hide)
+    )
+    (property "Datasheet" "" (at 97.79 129.54 0)
+      (effects (font (size 1.27 1.27)) hide)
+    )
+    (property "SNAPEDA_PACKAGE_ID" "25043" (at 97.79 129.54 0)
+      (effects (font (size 1.27 1.27)) (justify bottom) hide)
+    )
+    (property "MAXIMUM_PACKAGE_HEIGHT" "9.6 mm" (at 97.79 129.54 0)
+      (effects (font (size 1.27 1.27)) (justify bottom) hide)
+    )
+    (property "STANDARD" "Manufacturer Recommendations" (at 97.79 129.54 0)
+      (effects (font (size 1.27 1.27)) (justify bottom) hide)
+    )
+    (property "PARTREV" "V.9A" (at 97.79 129.54 0)
+      (effects (font (size 1.27 1.27)) (justify bottom) hide)
+    )
+    (property "MANUFACTURER" "Kingbright" (at 97.79 129.54 0)
+      (effects (font (size 1.27 1.27)) (justify bottom) hide)
+    )
+    (property "SNAPEDA_PN" "WP154A4SUREQBFZGC" (at 97.79 129.54 0)
+      (effects (font (size 1.27 1.27)) (justify bottom) hide)
+    )
+    (pin "1")
+    (pin "2")
+    (pin "3")
+    (pin "4")
+    (instances
+      (project "ROSE-PILK_v1"
+        (path "/3dfb9737-68ba-4ca9-8085-72e4f57f9e50/210ab0c2-9b77-4742-8f85-c7730efc701e/6e0de894-925c-49de-9455-676e538ebb3b"
+          (reference "D18") (unit 1)
+        )
+      )
     )
   )
