File: noname-board/ROSE-PILK_v1.5/Power_Connectors.kicad_sch (KiCad schematic)
At the start: 6 parts, among them J12 Conn_02x08_Counter_Clockwise, J13 Conn_02x08_Counter_Clockwise, J14 Conn_02x08_Counter_Clockwise, J15 Conn_02x08_Counter_Clockwise, J18 Conn_02x08_Counter_Clockwise, J19 Conn_02x08_Counter_Clockwise

Commit message: changez
Parts:
- removed J15, J18: Conn_02x08_Counter_Clockwise, Connector_PinSocket_2.00mm:PinSocket_2x08_P2.00mm_Vertical, symbol Connector_Generic:Conn_02x08_Counter_Clockwise
