File: noname-board/ROSE-PILK_v1.5/RP2040-Connect.kicad_sch (KiCad schematic)
At the start: 8 parts

Commit message: changez
Parts:
- removed R48, R49, R50, R51, R52, R53: 0, Resistor_THT:R_Axial_DIN0207_L6.3mm_D2.5mm_P10.16mm_Horizontal, symbol Device:R
Connections:
- net GPIO2-A is gone; now on net GPIO0-A: R46.1
- net GPIO3-A is gone; now on net GPIO1-A: R47.1
- net SWCLK-B is gone; now on net GPIO1-B: R46.2
- net SWDIO-B is gone; now on net GPIO0-B: R47.2
Other:
- note removed: "A as Master"
- note removed: "B as Master"
Changed lines of the file:
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@@
 (kicad_sch (version 20230121) (generator eeschema)
   (paper "A4")
-  (wire (pts (xy 114.3 34.29) (xy 116.84 34.29))
-    (stroke (width 0) (type default))
-  )
-  (wire (pts (xy 124.46 34.29) (xy 127 34.29))
-    (stroke (width 0) (type default))
-  )
-  (wire (pts (xy 60.96 62.23) (xy 63.5 62.23))
-    (stroke (width 0) (type default))
-  )
-  (wire (pts (xy 114.3 62.23) (xy 116.84 62.23))
-    (stroke (width 0) (type default))
-  )
   (wire (pts (xy 71.12 44.45) (xy 73.66 44.45))
-    (stroke (width 0) (type default))
-  )
-  (wire (pts (xy 114.3 44.45) (xy 116.84 44.45))
-    (stroke (width 0) (type default))
-  )
-  (wire (pts (xy 114.3 53.34) (xy 116.84 53.34))
-    (stroke (width 0) (type default))
-  )
-  (wire (pts (xy 124.46 53.34) (xy 127 53.34))
     (stroke (width 0) (type default))
   )
@@
     (stroke (width 0) (type default))
   )
-  (wire (pts (xy 71.12 53.34) (xy 73.66 53.34))
-    (stroke (width 0) (type default))
-  )
   (wire (pts (xy 60.96 34.29) (xy 63.5 34.29))
-    (stroke (width 0) (type default))
-  )
-  (wire (pts (xy 124.46 44.45) (xy 127 44.45))
-    (stroke (width 0) (type default))
-  )
-  (wire (pts (xy 71.12 62.23) (xy 73.66 62.23))
     (stroke (width 0) (type default))
   )
@@
     (stroke (width 0) (type default))
   )
-  (wire (pts (xy 60.96 53.34) (xy 63.5 53.34))
-    (stroke (width 0) (type default))
-  )
-  (wire (pts (xy 124.46 62.23) (xy 127 62.23))
-    (stroke (width 0) (type default))
-  )
-  (text "A as Master" (at 63.5 25.4 0)
-    (effects (font (size 1.27 1.27)) (justify left bottom))
-  )
-  (text "B as Master" (at 114.3 24.13 0)
-    (effects (font (size 1.27 1.27)) (justify left bottom))
-  )
-  (hierarchical_label "GPIO3-B" (shape input) (at 114.3 44.45 180) (fields_autoplaced)
+  (hierarchical_label "GPIO0-A" (shape input) (at 60.96 34.29 180) (fields_autoplaced)
     (effects (font (size 1.27 1.27)) (justify right))
   )
-  (hierarchical_label "GPIO2-A" (shape input) (at 60.96 34.29 180) (fields_autoplaced)
+  (hierarchical_label "GPIO1-A" (shape input) (at 60.96 44.45 180) (fields_autoplaced)
     (effects (font (size 1.27 1.27)) (justify right))
   )
-  (hierarchical_label "GPIO1-A" (shape input) (at 127 53.34 0) (fields_autoplaced)
+  (hierarchical_label "GPIO1-B" (shape input) (at 73.66 34.29 0) (fields_autoplaced)
     (effects (font (size 1.27 1.27)) (justify left))
   )
-  (hierarchical_label "GPIO1-B" (shape input) (at 73.66 53.34 0) (fields_autoplaced)
+  (hierarchical_label "GPIO0-B" (shape input) (at 73.66 44.45 0) (fields_autoplaced)
     (effects (font (size 1.27 1.27)) (justify left))
-  )
-  (hierarchical_label "GPIO5-A" (shape input) (at 60.96 62.23 180) (fields_autoplaced)
-    (effects (font (size 1.27 1.27)) (justify right))
-  )
-  (hierarchical_label "GPIO0-B" (shape input) (at 73.66 62.23 0) (fields_autoplaced)
-    (effects (font (size 1.27 1.27)) (justify left))
-  )
-  (hierarchical_label "GPIO3-A" (shape input) (at 60.96 44.45 180) (fields_autoplaced)
-    (effects (font (size 1.27 1.27)) (justify right))
-  )
-  (hierarchical_label "SWDIO-A" (shape input) (at 127 44.45 0) (fields_autoplaced)
-    (effects (font (size 1.27 1.27)) (justify left))
-  )
-  (hierarchical_label "SWCLK-A" (shape input) (at 127 34.29 0) (fields_autoplaced)
-    (effects (font (size 1.27 1.27)) (justify left))
-  )
-  (hierarchical_label "GPIO4-B" (shape input) (at 114.3 53.34 180) (fields_autoplaced)
-    (effects (font (size 1.27 1.27)) (justify right))
-  )
-  (hierarchical_label "SWCLK-B" (shape input) (at 73.66 34.29 0) (fields_autoplaced)
-    (effects (font (size 1.27 1.27)) (justify left))
-  )
-  (hierarchical_label "GPIO4-A" (shape input) (at 60.96 53.34 180) (fields_autoplaced)
-    (effects (font (size 1.27 1.27)) (justify right))
-  )
-  (hierarchical_label "SWDIO-B" (shape input) (at 73.66 44.45 0) (fields_autoplaced)
-    (effects (font (size 1.27 1.27)) (justify left))
-  )
-  (hierarchical_label "GPIO0-A" (shape input) (at 127 62.23 0) (fields_autoplaced)
-    (effects (font (size 1.27 1.27)) (justify left))
-  )
-  (hierarchical_label "GPIO2-B" (shape input) (at 114.3 34.29 180) (fields_autoplaced)
-    (effects (font (size 1.27 1.27)) (justify right))
-  )
-  (hierarchical_label "GPIO5-B" (shape input) (at 114.3 62.23 180) (fields_autoplaced)
-    (effects (font (size 1.27 1.27)) (justify right))
-  )
-  (symbol (lib_id "Device:R") (at 120.65 44.45 90) (unit 1)
-    (in_bom yes) (on_board yes) (dnp no)
-    (property "Reference" "R51" (at 120.65 39.37 90)
-      (effects (font (size 1.27 1.27)))
-    )
-    (property "Value" "0" (at 120.65 41.91 90)
-      (effects (font (size 1.27 1.27)))
-    )
-    (property "Footprint" "Resistor_THT:R_Axial_DIN0207_L6.3mm_D2.5mm_P10.16mm_Horizontal" (at 120.65 46.228 90)
-      (effects (font (size 1.27 1.27)) hide)
-    )
-    (property "Datasheet" "~" (at 120.65 44.45 0)
-      (effects (font (size 1.27 1.27)) hide)
-    )
-    (pin "1")
-    (pin "2")
-    (instances
-      (project "ROSE-PILK_v1"
-        (path "/3dfb9737-68ba-4ca9-8085-72e4f57f9e50/47bf5c44-9f46-40eb-9079-d0aa3a0f2164"
-          (reference "R51") (unit 1)
-        )
-      )
-    )
-  )
-  (symbol (lib_id "Device:R") (at 120.65 34.29 90) (unit 1)
-    (in_bom yes) (on_board yes) (dnp no)
-    (property "Reference" "R50" (at 120.65 29.21 90)
-      (effects (font (size 1.27 1.27)))
-    )
-    (property "Value" "0" (at 120.65 31.75 90)
-      (effects (font (size 1.27 1.27)))
-    )
-    (property "Footprint" "Resistor_THT:R_Axial_DIN0207_L6.3mm_D2.5mm_P10.16mm_Horizontal" (at 120.65 36.068 90)
-      (effects (font (size 1.27 1.27)) hide)
-    )
-    (property "Datasheet" "~" (at 120.65 34.29 0)
-      (effects (font (size 1.27 1.27)) hide)
-    )
-    (pin "1")
-    (pin "2")
-    (instances
-      (project "ROSE-PILK_v1"
-        (path "/3dfb9737-68ba-4ca9-8085-72e4f57f9e50/47bf5c44-9f46-40eb-9079-d0aa3a0f2164"
-          (reference "R50") (unit 1)
-        )
-      )
-    )
   )
   (symbol (lib_id "Device:R") (at 67.31 34.29 90) (unit 1)
@@
         (path "/3dfb9737-68ba-4ca9-8085-72e4f57f9e50/47bf5c44-9f46-40eb-9079-d0aa3a0f2164"
           (reference "R46") (unit 1)
-        )
-      )
-    )
-  )
-  (symbol (lib_id "Device:R") (at 67.31 53.34 90) (unit 1)
-    (in_bom yes) (on_board yes) (dnp no)
-    (property "Reference" "R48" (at 67.31 48.26 90)
-      (effects (font (size 1.27 1.27)))
-    )
-    (property "Value" "0" (at 67.31 50.8 90)
-      (effects (font (size 1.27 1.27)))
-    )
-    (property "Footprint" "Resistor_THT:R_Axial_DIN0207_L6.3mm_D2.5mm_P10.16mm_Horizontal" (at 67.31 55.118 90)
-      (effects (font (size 1.27 1.27)) hide)
-    )
-    (property "Datasheet" "~" (at 67.31 53.34 0)
-      (effects (font (size 1.27 1.27)) hide)
-    )
-    (pin "1")
-    (pin "2")
-    (instances
-      (project "ROSE-PILK_v1"
-        (path "/3dfb9737-68ba-4ca9-8085-72e4f57f9e50/47bf5c44-9f46-40eb-9079-d0aa3a0f2164"
-          (reference "R48") (unit 1)
-        )
-      )
-    )
-  )
-  (symbol (lib_id "Device:R") (at 120.65 53.34 90) (unit 1)
-    (in_bom yes) (on_board yes) (dnp no)
-    (property "Reference" "R52" (at 120.65 48.26 90)
-      (effects (font (size 1.27 1.27)))
-    )
-    (property "Value" "0" (at 120.65 50.8 90)
-      (effects (font (size 1.27 1.27)))
-    )
-    (property "Footprint" "Resistor_THT:R_Axial_DIN0207_L6.3mm_D2.5mm_P10.16mm_Horizontal" (at 120.65 55.118 90)
-      (effects (font (size 1.27 1.27)) hide)
-    )
-    (property "Datasheet" "~" (at 120.65 53.34 0)
-      (effects (font (size 1.27 1.27)) hide)
-    )
-    (pin "1")
-    (pin "2")
-    (instances
-      (project "ROSE-PILK_v1"
-        (path "/3dfb9737-68ba-4ca9-8085-72e4f57f9e50/47bf5c44-9f46-40eb-9079-d0aa3a0f2164"
-          (reference "R52") (unit 1)
-        )
-      )
-    )
-  )
-  (symbol (lib_id "Device:R") (at 120.65 62.23 90) (unit 1)
-    (in_bom yes) (on_board yes) (dnp no)
-    (property "Reference" "R53" (at 120.65 57.15 90)
-      (effects (font (size 1.27 1.27)))
-    )
-    (property "Value" "0" (at 120.65 59.69 90)
-      (effects (font (size 1.27 1.27)))
-    )
-    (property "Footprint" "Resistor_THT:R_Axial_DIN0207_L6.3mm_D2.5mm_P10.16mm_Horizontal" (at 120.65 64.008 90)
-      (effects (font (size 1.27 1.27)) hide)
-    )
-    (property "Datasheet" "~" (at 120.65 62.23 0)
-      (effects (font (size 1.27 1.27)) hide)
-    )
-    (pin "1")
-    (pin "2")
-    (instances
-      (project "ROSE-PILK_v1"
-        (path "/3dfb9737-68ba-4ca9-8085-72e4f57f9e50/47bf5c44-9f46-40eb-9079-d0aa3a0f2164"
-          (reference "R53") (unit 1)
         )
       )
@@
         )
       )
-    )
-  )
-  (symbol (lib_id "Device:R") (at 67.31 62.23 90) (unit 1)
-    (in_bom yes) (on_board yes) (dnp no)
-    (property "Reference" "R49" (at 67.31 57.15 90)
-      (effects (font (size 1.27 1.27)))
-    )
-    (property "Value" "0" (at 67.31 59.69 90)
-      (effects (font (size 1.27 1.27)))
-    )
-    (property "Footprint" "Resistor_THT:R_Axial_DIN0207_L6.3mm_D2.5mm_P10.16mm_Horizontal" (at 67.31 64.008 90)
-      (effects (font (size 1.27 1.27)) hide)
-    )
-    (property "Datasheet" "~" (at 67.31 62.23 0)
-      (effects (font (size 1.27 1.27)) hide)
-    )
-    (pin "1")
-    (pin "2")
-    (instances
-      (project "ROSE-PILK_v1"
-        (path "/3dfb9737-68ba-4ca9-8085-72e4f57f9e50/47bf5c44-9f46-40eb-9079-d0aa3a0f2164"
-          (reference "R49") (unit 1)
-        )
-      )
