File: noname-board/ROSE-PILK_v1.5/power.kicad_sch (KiCad schematic)
At the start: 14 parts, among them J10 Conn_01x01_Pin, J8 Conn_01x01_Pin, J9 Conn_01x01_Pin, Q1 LM2940CT-5.0_NOPB, U11 RT6150B-33GQW, U4 XT30UPB-M

Commit message: Big changes
Parts:
- removed C1, C4: 47uF, Capacitor_THT:C_Disc_D7.0mm_W2.5mm_P5.00mm, symbol Device:C
- removed D16: 1N5817, Diode_THT:D_DO-41_SOD81_P10.16mm_Horizontal, symbol Diode:1N5817
- removed J10, J8, J9: Conn_01x01_Pin, Connector_PinSocket_1.27mm:PinSocket_1x01_P1.27mm_Vertical, symbol Connector:Conn_01x01_Pin
- removed L1: 2.2uH, Capacitor_THT:CP_Radial_D5.0mm_P2.00mm, symbol Device:L
- removed R1: 100K, Resistor_THT:R_Axial_DIN0207_L6.3mm_D2.5mm_P10.16mm_Horizontal, symbol Device:R
- removed U11: RT6150B-33GQW, RT6150B:SON50P250X250X80-11N, symbol RT6150B:RT6150B-33GQW
Other:
- note removed: "PS"
- note removed: "V_BUS"
- note removed: "V_SYS"
