File: noname-board/ROSE-PILK_v1.5/GPIO_Connect.kicad_sch (KiCad schematic)
At the start: 2 parts, among them J11 Conn_02x24_Odd_Even, J17 Conn_02x09_Odd_Even

Commit message: I changed things shit my bad
Parts:
- J11: footprint Connector_PinHeader_2.00mm:PinHeader_2x24_P2.00mm_Vertical -> Connector_PinSocket_2.00mm:PinSocket_2x24_P2.00mm_Vertical
- J17: footprint Connector_PinHeader_2.00mm:PinHeader_2x09_P2.00mm_Vertical -> Connector_PinSocket_2.00mm:PinSocket_2x09_P2.00mm_Vertical
Changed lines of the file:
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@@
       (effects (font (size 1.27 1.27)))
     )
-    (property "Footprint" "Connector_PinHeader_2.00mm:PinHeader_2x09_P2.00mm_Vertical" (at 53.34 96.52 0)
+    (property "Footprint" "Connector_PinSocket_2.00mm:PinSocket_2x09_P2.00mm_Vertical" (at 53.34 96.52 0)
       (effects (font (size 1.27 1.27)) hide)
     )
@@
       (effects (font (size 1.27 1.27)))
     )
-    (property "Footprint" "Connector_PinHeader_2.00mm:PinHeader_2x24_P2.00mm_Vertical" (at 191.77 88.9 0)
+    (property "Footprint" "Connector_PinSocket_2.00mm:PinSocket_2x24_P2.00mm_Vertical" (at 191.77 88.9 0)
       (effects (font (size 1.27 1.27)) hide)
     )

Commit message: TRACING PLACING AND OTHER SHIT I CAN'T BE BOTHERED DESCRIBING
Parts:
- removed J11: Conn_02x24_Odd_Even, Connector_PinSocket_2.00mm:PinSocket_2x24_P2.00mm_Vertical, symbol Connector_Generic:Conn_02x24_Odd_Even
- removed J17: Conn_02x09_Odd_Even, Connector_PinSocket_2.00mm:PinSocket_2x09_P2.00mm_Vertical, symbol Connector_Generic:Conn_02x09_Odd_Even
- added J8: Conn_02x06_Counter_Clockwise, Connector_PinSocket_2.00mm:PinSocket_2x06_P2.00mm_Vertical, symbol Connector_Generic:Conn_02x06_Counter_Clockwise
Connections:
- net A_GPIO26: now also J8.3 (Pin_3)
- net A_GPIO27: now also J8.4 (Pin_4)
- net A_GPIO28: now also J8.5 (Pin_5)
- net B_GPIO12: now also J8.11 (Pin_11)
- net B_GPIO13: now also J8.10 (Pin_10)
- net B_GPIO14: now also J8.9 (Pin_9)
- net B_GPIO26: now also J8.8 (Pin_8)
- net B_GPIO27: now also J8.7 (Pin_7)
- net B_GPIO28: now also J8.6 (Pin_6)
- net B_GPIO8: now also J8.12 (Pin_12)
- new net A_GPIO21: J8.1 (Pin_1)
- new net A_GPIO22: J8.2 (Pin_2)
