File: noname-board/ROSE-PILK_v1.5/CAN2.kicad_sch (KiCad schematic)
At the start: 3 parts, among them J4 Conn_01x04, U5 SN65HVD230DR

Commit message: TRACING PLACING AND OTHER SHIT I CAN'T BE BOTHERED DESCRIBING
Parts:
- added J6: Conn_01x04, Connector_JST:JST_GH_SM04B-GHS-TB_1x04-1MP_P1.25mm_Horizontal, symbol Connector_Generic:Conn_01x04
- J4: footprint SM04B_GHS_TB_LF__SN__:JST_SM04B-GHS-TB_LF__SN_- -> Connector_JST:JST_GH_SM04B-GHS-TB_1x04-1MP_P1.25mm_Horizontal
Connections:
- net 5V: now also J6.4 (Pin_4)
- net GND: now also J6.3 (Pin_3)
- net at J4.1 (Pin_1), R32.2, U5.6 (CANL): now also J6.1 (Pin_1)
- net at J4.2 (Pin_2), R32.1, U5.7 (CANH): now also J6.2 (Pin_2)
Changed lines of the file:
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@@
   (junction (at 179.07 82.55) (diameter 0) (color 0 0 0 0)
+  )
+  (junction (at 189.23 82.55) (diameter 0) (color 0 0 0 0)
+  )
+  (junction (at 187.96 90.17) (diameter 0) (color 0 0 0 0)
   )
   (no_connect (at 160.02 90.17))
@@
     (stroke (width 0) (type default))
   )
-  (wire (pts (xy 179.07 82.55) (xy 190.5 82.55))
+  (wire (pts (xy 179.07 82.55) (xy 189.23 82.55))
     (stroke (width 0) (type default))
   )
@@
   )
   (wire (pts (xy 201.93 87.63) (xy 190.5 87.63))
+    (stroke (width 0) (type default))
+  )
+  (wire (pts (xy 201.93 105.41) (xy 187.96 105.41))
+    (stroke (width 0) (type default))
+  )
+  (wire (pts (xy 201.93 102.87) (xy 189.23 102.87))
     (stroke (width 0) (type default))
   )
@@
     (stroke (width 0) (type default))
   )
-  (wire (pts (xy 179.07 90.17) (xy 201.93 90.17))
+  (wire (pts (xy 179.07 90.17) (xy 187.96 90.17))
     (stroke (width 0) (type default))
   )
   (wire (pts (xy 97.79 82.55) (xy 104.14 82.55))
+    (stroke (width 0) (type default))
+  )
+  (wire (pts (xy 187.96 90.17) (xy 201.93 90.17))
     (stroke (width 0) (type default))
   )
@@
     (stroke (width 0) (type default))
   )
+  (wire (pts (xy 189.23 82.55) (xy 190.5 82.55))
+    (stroke (width 0) (type default))
+  )
+  (wire (pts (xy 187.96 105.41) (xy 187.96 90.17))
+    (stroke (width 0) (type default))
+  )
+  (wire (pts (xy 189.23 102.87) (xy 189.23 82.55))
+    (stroke (width 0) (type default))
+  )
   (text "CAN_H\n" (at 190.5 87.63 0)
     (effects (font (size 1.27 1.27)) (justify left bottom))
@@
   (text "CAN_L" (at 190.5 92.71 0)
     (effects (font (size 1.27 1.27)) (justify left bottom))
+  )
+  (hierarchical_label "GND" (shape input) (at 201.93 100.33 180) (fields_autoplaced)
+    (effects (font (size 1.27 1.27)) (justify right))
   )
   (hierarchical_label "GND" (shape input) (at 97.79 85.09 180) (fields_autoplaced)
@@
     (effects (font (size 1.27 1.27)) (justify right))
   )
+  (hierarchical_label "5V" (shape input) (at 201.93 97.79 180) (fields_autoplaced)
+    (effects (font (size 1.27 1.27)) (justify right))
+  )
   (hierarchical_label "3V3" (shape input) (at 97.79 87.63 180) (fields_autoplaced)
     (effects (font (size 1.27 1.27)) (justify right))
@@
   (hierarchical_label "GND" (shape input) (at 201.93 85.09 180) (fields_autoplaced)
     (effects (font (size 1.27 1.27)) (justify right))
+  )
+  (symbol (lib_id "Connector_Generic:Conn_01x04") (at 207.01 102.87 0) (mirror x) (unit 1)
+    (in_bom yes) (on_board yes) (dnp no)
+    (property "Reference" "J6" (at 209.55 102.87 0)
+      (effects (font (size 1.27 1.27)) (justify left))
+    )
+    (property "Value" "Conn_01x04" (at 209.55 100.33 0)
+      (effects (font (size 1.27 1.27)) (justify left))
+    )
+    (property "Footprint" "Connector_JST:JST_GH_SM04B-GHS-TB_1x04-1MP_P1.25mm_Horizontal" (at 207.01 102.87 0)
+      (effects (font (size 1.27 1.27)) hide)
+    )
+    (property "Datasheet" "~" (at 207.01 102.87 0)
+      (effects (font (size 1.27 1.27)) hide)
+    )
+    (pin "1")
+    (pin "2")
+    (pin "3")
+    (pin "4")
+    (instances
+      (project "ROSE-PILK_v1"
+        (path "/3dfb9737-68ba-4ca9-8085-72e4f57f9e50/cc566290-d472-48a8-a9ae-4e54f87660da"
+          (reference "J6") (unit 1)
+        )
+      )
+    )
   )
   (symbol (lib_id "SN65HVD230DR:SN65HVD230DR") (at 104.14 82.55 0) (unit 1)
@@
       (effects (font (size 1.27 1.27)) (justify left))
     )
-    (property "Footprint" "SM04B_GHS_TB_LF__SN__:JST_SM04B-GHS-TB_LF__SN_-" (at 207.01 87.63 0)
+    (property "Footprint" "Connector_JST:JST_GH_SM04B-GHS-TB_1x04-1MP_P1.25mm_Horizontal" (at 207.01 87.63 0)
       (effects (font (size 1.27 1.27)) hide)
     )

Commit message: Tracing part 2
Parts:
- added C1: .1uF, Capacitor_THT:C_Disc_D7.0mm_W2.5mm_P5.00mm, symbol Device:C
Connections:
- net 3V3: now also C1.1
- net GND: now also C1.2
Changed lines of the file:
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@@
   (junction (at 179.07 82.55) (diameter 0) (color 0 0 0 0)
   )
+  (junction (at 100.33 85.09) (diameter 0) (color 0 0 0 0)
+  )
   (junction (at 189.23 82.55) (diameter 0) (color 0 0 0 0)
   )
   (junction (at 187.96 90.17) (diameter 0) (color 0 0 0 0)
+  )
+  (junction (at 99.695 87.63) (diameter 0) (color 0 0 0 0)
   )
   (no_connect (at 160.02 90.17))
@@
     (stroke (width 0) (type default))
   )
+  (wire (pts (xy 74.93 81.915) (xy 100.33 81.915))
+    (stroke (width 0) (type default))
+  )
   (wire (pts (xy 201.93 102.87) (xy 189.23 102.87))
     (stroke (width 0) (type default))
@@
     (stroke (width 0) (type default))
   )
-  (wire (pts (xy 97.79 85.09) (xy 104.14 85.09))
+  (wire (pts (xy 97.79 85.09) (xy 100.33 85.09))
     (stroke (width 0) (type default))
   )
@@
     (stroke (width 0) (type default))
   )
+  (wire (pts (xy 99.695 87.63) (xy 104.14 87.63))
+    (stroke (width 0) (type default))
+  )
   (wire (pts (xy 179.07 90.17) (xy 187.96 90.17))
     (stroke (width 0) (type default))
@@
     (stroke (width 0) (type default))
   )
-  (wire (pts (xy 97.79 87.63) (xy 104.14 87.63))
+  (wire (pts (xy 97.79 87.63) (xy 99.695 87.63))
     (stroke (width 0) (type default))
   )
@@
     (stroke (width 0) (type default))
   )
+  (wire (pts (xy 100.33 81.915) (xy 100.33 85.09))
+    (stroke (width 0) (type default))
+  )
+  (wire (pts (xy 100.33 85.09) (xy 104.14 85.09))
+    (stroke (width 0) (type default))
+  )
   (wire (pts (xy 189.23 82.55) (xy 190.5 82.55))
     (stroke (width 0) (type default))
@@
   )
   (wire (pts (xy 189.23 102.87) (xy 189.23 82.55))
+    (stroke (width 0) (type default))
+  )
+  (wire (pts (xy 74.93 89.535) (xy 99.695 89.535))
+    (stroke (width 0) (type default))
+  )
+  (wire (pts (xy 99.695 89.535) (xy 99.695 87.63))
     (stroke (width 0) (type default))
   )
@@
         )
       )
+    )
+  )
+  (symbol (lib_id "Device:C") (at 74.93 85.725 180) (unit 1)
+    (in_bom yes) (on_board yes) (dnp no)
+    (property "Reference" "C1" (at 71.12 86.995 0)
+      (effects (font (size 1.27 1.27)) (justify left))
+    )
+    (property "Value" ".1uF" (at 71.12 84.455 0)
+      (effects (font (size 1.27 1.27)) (justify left))
+    )
+    (property "Footprint" "Capacitor_THT:C_Disc_D7.0mm_W2.5mm_P5.00mm" (at 73.9648 81.915 0)
+      (effects (font (size 1.27 1.27)) hide)
+    )
+    (property "Datasheet" "~" (at 74.93 85.725 0)
+      (effects (font (size 1.27 1.27)) hide)
+    )
+    (pin "1")
+    (pin "2")
+    (instances
+      (project "ROSE-PILK_v1"
+        (path "/3dfb9737-68ba-4ca9-8085-72e4f57f9e50"
+          (reference "C1") (unit 1)
+        )
+        (path "/3dfb9737-68ba-4ca9-8085-72e4f57f9e50/a50dd852-2d1e-4bb7-8a2f-4a12eba0cf9f"
+          (reference "C5") (unit 1)
+        )
+        (path "/3dfb9737-68ba-4ca9-8085-72e4f57f9e50/cc566290-d472-48a8-a9ae-4e54f87660da"
+          (reference "CAN2") (unit 1)
+        )
+      )
