File: noname-board/ROSE-PILK_v1.5/DR16.kicad_sch (KiCad schematic)
At the start: 4 parts, among them J2 Conn_01x03, Q3 PN2222A

Commit message: TRACING PLACING AND OTHER SHIT I CAN'T BE BOTHERED DESCRIBING
Connections:
- net USART RX renamed USART TX
Changed lines of the file:
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@@
     (effects (font (size 1.27 1.27)) (justify right))
   )
-  (hierarchical_label "USART RX" (shape input) (at 156.21 73.66 180) (fields_autoplaced)
+  (hierarchical_label "USART TX" (shape input) (at 156.21 73.66 180) (fields_autoplaced)
     (effects (font (size 1.27 1.27)) (justify right))
   )

Commit message: Tracing part 2
Parts:
- added C2: .1uF, Capacitor_THT:C_Disc_D7.0mm_W2.5mm_P5.00mm, symbol Device:C
Connections:
- net 5V: now also C2.2
- net GND: now also C2.1
Changed lines of the file:
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@@
   (junction (at 171.45 73.66) (diameter 0) (color 0 0 0 0)
+  )
+  (junction (at 149.86 99.06) (diameter 0) (color 0 0 0 0)
+  )
+  (junction (at 146.05 99.695) (diameter 0) (color 0 0 0 0)
   )
   (wire (pts (xy 156.21 73.66) (xy 171.45 73.66))
@@
   )
   (wire (pts (xy 171.45 71.12) (xy 171.45 73.66))
+    (stroke (width 0) (type default))
+  )
+  (wire (pts (xy 146.05 99.695) (xy 146.05 100.33))
     (stroke (width 0) (type default))
   )
@@
     (stroke (width 0) (type default))
   )
-  (wire (pts (xy 146.05 97.79) (xy 146.05 100.33))
+  (wire (pts (xy 146.05 97.79) (xy 146.05 99.695))
+    (stroke (width 0) (type default))
+  )
+  (wire (pts (xy 144.78 113.665) (xy 144.78 99.695))
     (stroke (width 0) (type default))
   )
@@
     (stroke (width 0) (type default))
   )
-  (wire (pts (xy 149.86 95.25) (xy 149.86 100.33))
+  (wire (pts (xy 149.86 95.25) (xy 149.86 99.06))
     (stroke (width 0) (type default))
   )
@@
     (stroke (width 0) (type default))
   )
+  (wire (pts (xy 144.78 99.695) (xy 146.05 99.695))
+    (stroke (width 0) (type default))
+  )
   (wire (pts (xy 171.45 73.66) (xy 171.45 87.63))
+    (stroke (width 0) (type default))
+  )
+  (wire (pts (xy 149.86 99.06) (xy 149.86 100.33))
+    (stroke (width 0) (type default))
+  )
+  (wire (pts (xy 152.4 113.665) (xy 152.4 99.06))
+    (stroke (width 0) (type default))
+  )
+  (wire (pts (xy 149.86 99.06) (xy 152.4 99.06))
     (stroke (width 0) (type default))
   )
@@
     (effects (font (size 1.27 1.27)) (justify right))
   )
+  (symbol (lib_id "Device:C") (at 148.59 113.665 90) (unit 1)
+    (in_bom yes) (on_board yes) (dnp no) (fields_autoplaced)
+    (property "Reference" "C2" (at 148.59 106.68 90)
+      (effects (font (size 1.27 1.27)))
+    )
+    (property "Value" ".1uF" (at 148.59 109.22 90)
+      (effects (font (size 1.27 1.27)))
+    )
+    (property "Footprint" "Capacitor_THT:C_Disc_D7.0mm_W2.5mm_P5.00mm" (at 152.4 112.6998 0)
+      (effects (font (size 1.27 1.27)) hide)
+    )
+    (property "Datasheet" "~" (at 148.59 113.665 0)
+      (effects (font (size 1.27 1.27)) hide)
+    )
+    (pin "1")
+    (pin "2")
+    (instances
+      (project "ROSE-PILK_v1"
+        (path "/3dfb9737-68ba-4ca9-8085-72e4f57f9e50/7f9280f8-5c56-426f-91c5-2013c74ffd42"
+          (reference "C2") (unit 1)
+        )
+        (path "/3dfb9737-68ba-4ca9-8085-72e4f57f9e50/c34ca0c5-7bce-4bc6-9986-6cfb64a47688"
+          (reference "DR16") (unit 1)
+        )
+      )
+      (project "power"
+        (path "/98742a09-6d32-4217-a474-ca7198a8eb01"
+          (reference "C1") (unit 1)
+        )
+        (path "/98742a09-6d32-4217-a474-ca7198a8eb01/5f1da244-199a-4c11-be94-62be443d4855"
+          (reference "C5") (unit 1)
+        )
+      )
+    )
+  )
   (symbol (lib_id "Device:R") (at 171.45 67.31 0) (unit 1)
