File: noname-board/ROSE-PILK_v1.5/QUAD.kicad_sch (KiCad schematic)
At the start: 2 parts, among them J1 Conn_01x04

Commit message: Tracing part 2
Parts:
- added QUAD1, QUAD2: .1uF, Capacitor_THT:C_Disc_D7.0mm_W2.5mm_P5.00mm, symbol Device:C
Connections:
- net 3V3: now also QUAD1.1, QUAD2.1
- net GND: now also QUAD1.2, QUAD2.2
Changed lines of the file:
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@@
 (kicad_sch (version 20230121) (generator eeschema)
   (paper "A4")
-  (wire (pts (xy 80.01 107.95) (xy 80.01 116.84))
+  (junction (at 80.01 113.665) (diameter 0) (color 0 0 0 0)
+  )
+  (junction (at 77.47 114.935) (diameter 0) (color 0 0 0 0)
+  )
+  (junction (at 69.85 53.975) (diameter 0) (color 0 0 0 0)
+  )
+  (junction (at 67.31 55.88) (diameter 0) (color 0 0 0 0)
+  )
+  (wire (pts (xy 80.01 107.95) (xy 80.01 113.665))
     (stroke (width 0) (type default))
   )
@@
     (stroke (width 0) (type default))
   )
-  (wire (pts (xy 67.31 49.53) (xy 67.31 58.42))
+  (wire (pts (xy 67.31 55.88) (xy 67.31 58.42))
+    (stroke (width 0) (type default))
+  )
+  (wire (pts (xy 67.31 49.53) (xy 67.31 55.88))
+    (stroke (width 0) (type default))
+  )
+  (wire (pts (xy 76.835 53.975) (xy 69.85 53.975))
+    (stroke (width 0) (type default))
+  )
+  (wire (pts (xy 86.36 113.665) (xy 80.01 113.665))
+    (stroke (width 0) (type default))
+  )
+  (wire (pts (xy 80.01 113.665) (xy 80.01 116.84))
+    (stroke (width 0) (type default))
+  )
+  (wire (pts (xy 77.47 114.935) (xy 77.47 116.84))
     (stroke (width 0) (type default))
   )
@@
     (stroke (width 0) (type default))
   )
-  (wire (pts (xy 77.47 107.95) (xy 77.47 116.84))
+  (wire (pts (xy 78.74 128.27) (xy 78.74 114.935))
+    (stroke (width 0) (type default))
+  )
+  (wire (pts (xy 69.215 69.85) (xy 69.215 55.88))
+    (stroke (width 0) (type default))
+  )
+  (wire (pts (xy 77.47 107.95) (xy 77.47 114.935))
     (stroke (width 0) (type default))
   )
@@
     (stroke (width 0) (type default))
   )
-  (wire (pts (xy 69.85 49.53) (xy 69.85 58.42))
+  (wire (pts (xy 69.85 49.53) (xy 69.85 53.975))
+    (stroke (width 0) (type default))
+  )
+  (wire (pts (xy 78.74 114.935) (xy 77.47 114.935))
+    (stroke (width 0) (type default))
+  )
+  (wire (pts (xy 86.36 128.27) (xy 86.36 113.665))
+    (stroke (width 0) (type default))
+  )
+  (wire (pts (xy 69.85 53.975) (xy 69.85 58.42))
+    (stroke (width 0) (type default))
+  )
+  (wire (pts (xy 69.215 55.88) (xy 67.31 55.88))
+    (stroke (width 0) (type default))
+  )
+  (wire (pts (xy 76.835 69.85) (xy 76.835 53.975))
     (stroke (width 0) (type default))
   )
@@
         )
       )
+    )
+  )
+  (symbol (lib_id "Device:C") (at 73.025 69.85 90) (unit 1)
+    (in_bom yes) (on_board yes) (dnp no) (fields_autoplaced)
+    (property "Reference" "QUAD1" (at 73.025 62.23 90)
+      (effects (font (size 1.27 1.27)))
+    )
+    (property "Value" ".1uF" (at 73.025 64.77 90)
+      (effects (font (size 1.27 1.27)))
+    )
+    (property "Footprint" "Capacitor_THT:C_Disc_D7.0mm_W2.5mm_P5.00mm" (at 76.835 68.8848 0)
+      (effects (font (size 1.27 1.27)) hide)
+    )
+    (property "Datasheet" "~" (at 73.025 69.85 0)
+      (effects (font (size 1.27 1.27)) hide)
+    )
+    (pin "1")
+    (pin "2")
+    (instances
+      (project "ROSE-PILK_v1"
+        (path "/3dfb9737-68ba-4ca9-8085-72e4f57f9e50/8e9d615d-761b-441b-83a7-0b32546be700"
+          (reference "QUAD1") (unit 1)
+        )
+      )
+    )
+  )
+  (symbol (lib_id "Device:C") (at 82.55 128.27 90) (unit 1)
+    (in_bom yes) (on_board yes) (dnp no) (fields_autoplaced)
+    (property "Reference" "QUAD2" (at 82.55 120.65 90)
+      (effects (font (size 1.27 1.27)))
+    )
+    (property "Value" ".1uF" (at 82.55 123.19 90)
+      (effects (font (size 1.27 1.27)))
+    )
+    (property "Footprint" "Capacitor_THT:C_Disc_D7.0mm_W2.5mm_P5.00mm" (at 86.36 127.3048 0)
+      (effects (font (size 1.27 1.27)) hide)
+    )
+    (property "Datasheet" "~" (at 82.55 128.27 0)
+      (effects (font (size 1.27 1.27)) hide)
+    )
+    (pin "1")
+    (pin "2")
+    (instances
+      (project "ROSE-PILK_v1"
+        (path "/3dfb9737-68ba-4ca9-8085-72e4f57f9e50/8e9d615d-761b-441b-83a7-0b32546be700"
+          (reference "QUAD2") (unit 1)
+        )
+      )
