File: noname-board/ROSE-PILK_v1.5 - Anthony/DR16.kicad_sch (KiCad schematic)
At the start: 5 parts, among them J2 Conn_01x03, Q3 PN2222A

Commit message: ahhhhh
Parts:
- R30, R31: value R -> 5k
Changed lines of the file:
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@@
       (effects (font (size 1.27 1.27)) (justify left))
     )
-    (property "Value" "R" (at 173.99 68.58 0)
+    (property "Value" "5k" (at 173.99 68.58 0)
       (effects (font (size 1.27 1.27)) (justify left))
     )
@@
       (effects (font (size 1.27 1.27)))
     )
-    (property "Value" "R" (at 157.48 88.9 90)
+    (property "Value" "5k" (at 157.48 88.9 90)
       (effects (font (size 1.27 1.27)))
     )
