File: noname-board/ROSE-PILK_v1.5 - Anthony/ROSE-PILK_v1.kicad_pcb (KiCad board)
At the start: 4 copper layers, 65 x 90 mm, 55 parts, among them J1 Conn_01x04, J10 Conn_02x09_Counter_Clockwise, J11 Conn_01x04, J12 Conn_02x02_Counter_Clockwise, J13 Conn_02x02_Counter_Clockwise, J2 Conn_01x03, J3 Conn_01x02, J4 Conn_01x04, J5 Conn_01x02, J6 Conn_01x04, J7 Conn_01x04, J9 Conn_01x03, Q1 LM2940CT-5.0_NOPB, Q3 PN2222A, SW1 SW_Push, SW2 SW_Push, U1 Pico A, U2 TXS0108EPW, U4 XT30UPB-M, U5 SN65HVD230DR, U6 Pico B, U7 SN65HVD230DR

Commit message: tweaks
Routing:
- net Net-(J1-Pin_3): track 45.8 -> 44.8 mm
- net Net-(J1-Pin_2): track 50.9 -> 50.2 mm
- net /3V3: track 256.1 -> 255.5 mm

Commit message: cleaned up a tid
Routing:
- net /P2P_2: track 78.8 -> 77.0 mm
- net Net-(D16-Pad3): track 49.1 -> 48.1 mm
- net /B3: track 62.7 -> 62.0 mm
Other:
- board text added: "Luci is a poopy head"

Commit message: t
Routing:
- net /A0: track 54.0 -> 55.3 mm
- net /A1: track 54.5 -> 55.6 mm
- net /SERVO: track 66.7 -> 65.7 mm
- net /A27: track 32.7 -> 33.6 mm
- net /CAN2_RX: track 44.9 -> 44.3 mm
- net /B5: track 45.1 -> 45.7 mm

Commit message: twkz
Routing:
- net Net-(D16-Pad1): track 51.3 -> 50.7 mm
Changed lines of the file:
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@@
   (segment (start 189.614009 86.375) (end 187.825 88.164009) (width 0.25) (layer "F.Cu") (net 30))
   (via (at 197.2 86.05) (size 0.8) (drill 0.4) (layers "F.Cu" "B.Cu") (net 30))
-  (segment (start 202.13 87) (end 206.63 82.5) (width 0.25) (layer "B.Cu") (net 30))
-  (segment (start 197.2 86.05) (end 198.15 87) (width 0.25) (layer "B.Cu") (net 30))
-  (segment (start 198.15 87) (end 202.13 87) (width 0.25) (layer "B.Cu") (net 30))
+  (segment (start 197.2 86.05) (end 197.75 86.6) (width 0.25) (layer "B.Cu") (net 30))
+  (segment (start 197.75 86.6) (end 202.53 86.6) (width 0.25) (layer "B.Cu") (net 30))
+  (segment (start 202.53 86.6) (end 206.63 82.5) (width 0.25) (layer "B.Cu") (net 30))
   (segment (start 188.955 94.965991) (end 191.225 97.235991) (width 0.25) (layer "F.Cu") (net 31))
   (segment (start 188.9995 92) (end 188.725 92) (width 0.25) (layer "F.Cu") (net 31))
@@
   (segment (start 191.225 114.855) (end 190.08 116) (width 0.25) (layer "F.Cu") (net 31))
   (via (at 188.9995 92) (size 0.8) (drill 0.4) (layers "F.Cu" "B.Cu") (net 31))
+  (segment (start 192.386509 87.1025) (end 204.5675 87.1025) (width 0.25) (layer "B.Cu") (net 31))
   (segment (start 188.955 91.9555) (end 188.955 90.534009) (width 0.25) (layer "B.Cu") (net 31))
-  (segment (start 195.699695 87.725) (end 203.945 87.725) (width 0.25) (layer "B.Cu") (net 31))
+  (segment (start 188.955 90.534009) (end 192.386509 87.1025) (width 0.25) (layer "B.Cu") (net 31))
+  (segment (start 204.5675 87.1025) (end 209.17 82.5) (width 0.25) (layer "B.Cu") (net 31))
   (segment (start 188.9995 92) (end 188.955 91.9555) (width 0.25) (layer "B.Cu") (net 31))
-  (segment (start 195.077195 87.1025) (end 195.699695 87.725) (width 0.25) (layer "B.Cu") (net 31))
-  (segment (start 188.955 90.534009) (end 192.386509 87.1025) (width 0.25) (layer "B.Cu") (net 31))
-  (segment (start 192.386509 87.1025) (end 195.077195 87.1025) (width 0.25) (layer "B.Cu") (net 31))
-  (segment (start 203.945 87.725) (end 209.17 82.5) (width 0.25) (layer "B.Cu") (net 31))
   (segment (start 168.61 123.545) (end 168.61 125.61) (width 0.25) (layer "F.Cu") (net 59))
   (segment (start 168 122.935) (end 168.61 123.545) (width 0.25) (layer "F.Cu") (net 59))
@@
   (segment (start 177.4505 111.290078) (end 177.4505 111.801491) (width 0.25) (layer "B.Cu") (net 89))
   (segment (start 200.71 122.55) (end 202.88 124.72) (width 0.25) (layer "B.Cu") (net 89))
+  (segment (start 198 110.557637) (end 198 114.5) (width 0.25) (layer "B.Cu") (net 90))
+  (segment (start 205.875 119.875) (end 205.875 121.92) (width 0.25) (layer "B.Cu") (net 90))
+  (segment (start 209.21 123.91) (end 209.21 125.32) (width 0.25) (layer "B.Cu") (net 90))
+  (segment (start 187.925 100.652387) (end 188.847613 101.575) (width 0.25) (layer "B.Cu") (net 90))
+  (segment (start 207.5 123.545) (end 208.845 123.545) (width 0.25) (layer "B.Cu") (net 90))
+  (segment (start 201.62 126) (end 200.34 124.72) (width 0.25) (layer "B.Cu") (net 90))
+  (segment (start 188.847613 101.575) (end 189.017363 101.575) (width 0.25) (layer "B.Cu") (net 90))
+  (segment (start 189.017363 101.575) (end 198 110.557637) (width 0.25) (layer "B.Cu") (net 90))
+  (segment (start 185.013604 96.65) (end 187.925 99.561396) (width 0.25) (layer "B.Cu") (net 90))
+  (segment (start 208.845 123.545) (end 209.21 123.91) (width 0.25) (layer "B.Cu") (net 90))
   (segment (start 174 98) (end 175.35 96.65) (width 0.25) (layer "B.Cu") (net 90))
+  (segment (start 199.7 116.2) (end 202.2 116.2) (width 0.25) (layer "B.Cu") (net 90))
   (segment (start 208.53 126) (end 201.62 126) (width 0.25) (layer "B.Cu") (net 90))
+  (segment (start 209.21 125.32) (end 208.53 126) (width 0.25) (layer "B.Cu") (net 90))
+  (segment (start 202.2 116.2) (end 205.875 119.875) (width 0.25) (layer "B.Cu") (net 90))
+  (segment (start 175.35 96.65) (end 185.013604 96.65) (width 0.25) (layer "B.Cu") (net 90))
+  (segment (start 187.925 99.561396) (end 187.925 100.652387) (width 0.25) (layer "B.Cu") (net 90))
+  (segment (start 198 114.5) (end 199.7 116.2) (width 0.25) (layer "B.Cu") (net 90))
   (segment (start 205.875 121.92) (end 207.5 123.545) (width 0.25) (layer "B.Cu") (net 90))
-  (segment (start 207.5 123.545) (end 208.845 123.545) (width 0.25) (layer "B.Cu") (net 90))
-  (segment (start 205.875 119.875) (end 205.875 121.92) (width 0.25) (layer "B.Cu") (net 90))
-  (segment (start 198.5 114.5) (end 200.48 116.48) (width 0.25) (layer "B.Cu") (net 90))
-  (segment (start 208.845 123.545) (end 209.21 123.91) (width 0.25) (layer "B.Cu") (net 90))
-  (segment (start 185.013604 96.65) (end 187.925 99.561396) (width 0.25) (layer "B.Cu") (net 90))
-  (segment (start 198.5 111.057637) (end 198.5 114.5) (width 0.25) (layer "B.Cu") (net 90))
-  (segment (start 175.35 96.65) (end 185.013604 96.65) (width 0.25) (layer "B.Cu") (net 90))
-  (segment (start 209.21 125.32) (end 208.53 126) (width 0.25) (layer "B.Cu") (net 90))
-  (segment (start 189.017363 101.575) (end 198.5 111.057637) (width 0.25) (layer "B.Cu") (net 90))
-  (segment (start 202.48 116.48) (end 205.875 119.875) (width 0.25) (layer "B.Cu") (net 90))
-  (segment (start 209.21 123.91) (end 209.21 125.32) (width 0.25) (layer "B.Cu") (net 90))
-  (segment (start 188.847613 101.575) (end 189.017363 101.575) (width 0.25) (layer "B.Cu") (net 90))
-  (segment (start 187.925 99.561396) (end 187.925 100.652387) (width 0.25) (layer "B.Cu") (net 90))
-  (segment (start 187.925 100.652387) (end 188.847613 101.575) (width 0.25) (layer "B.Cu") (net 90))
-  (segment (start 200.48 116.48) (end 202.48 116.48) (width 0.25) (layer "B.Cu") (net 90))
-  (segment (start 201.62 126) (end 200.34 124.72) (width 0.25) (layer "B.Cu") (net 90))
   (segment (start 170.5 112.2755) (end 170.5 99.5) (width 0.25) (layer "F.Cu") (net 91))
   (segment (start 170.2755 112.5) (end 170.5 112.2755) (width 0.25) (layer "F.Cu") (net 91))

Commit message: power hour
Connections:
- U4 pad P$2: Net-(D17-A) -> /GND
Changed lines of the file:
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@@
       (net 4 "Net-(Q1-IN)") (pinfunction "+") (pintype "passive") (solder_mask_margin 0.102))
     (pad "P$2" thru_hole circle (at 2.5 0) (size 2.7 2.7) (drill 1.8) (layers "*.Cu" "*.Mask")
-      (net 19 "Net-(D17-A)") (pinfunction "-") (pintype "passive") (solder_mask_margin 0.102))
+      (net 1 "/GND") (pinfunction "-") (pintype "passive") (solder_mask_margin 0.102))
   )
   (footprint "PS1024ALRED:SW_PS1024ALRED" (layer "F.Cu")
