File: 2024-25/Onboarding/kirschit/kirschit.kicad_sch (KiCad schematic)
At the start: 6 parts, among them J1 Conn_01x04, J2 Conn_01x02, SW1 SW_SPST, SW2 SW_SPST

Commit message: Finished schematic
Parts:
- removed J2: Conn_01x02, Connector_PinSocket_2.54mm:PinSocket_1x02_P2.54mm_Vertical, symbol Connector_Generic:Conn_01x02
- removed R2, R3: 330, Resistor_THT:R_Axial_DIN0309_L9.0mm_D3.2mm_P15.24mm_Horizontal, symbol Device:R
- added LEDR1: Conn_01x04, Connector_PinSocket_2.54mm:PinSocket_1x04_P2.54mm_Vertical, symbol Connector_Generic:Conn_01x04
- added Lion_Charger1: Conn_01x08, Connector_PinSocket_2.54mm:PinSocket_1x08_P2.54mm_Vertical, symbol Connector_Generic:Conn_01x08
- added SW3: EN, RB141C1100:SW_RB141C1100, symbol Switch:SW_SPST
- LEDL1: renamed from J1; footprint Connector_PinSocket_1.00mm:PinSocket_1x04_P1.00mm_Vertical -> Connector_PinSocket_2.54mm:PinSocket_1x04_P2.54mm_Vertical
- SW1: value SW_SPST -> LEDR; footprint Button_Switch_THT:SW_DIP_SPSTx01_Slide_6.7x4.1mm_W7.62mm_P2.54mm_LowProfile -> RB141C1100:SW_RB141C1100
- SW2: value SW_SPST -> LEDB; footprint Button_Switch_THT:SW_DIP_SPSTx01_Slide_6.7x4.1mm_W7.62mm_P2.54mm_LowProfile -> RB141C1100:SW_RB141C1100
Connections:
- net 5V: now also LEDR1.1 (Pin_1), Lion_Charger1.8 (Pin_8)
- net GND: now also Lion_Charger1.2 (Pin_2), Lion_Charger1.5 (Pin_5), Lion_Charger1.7 (Pin_7), SW3.2 (B)
- net LEDB: now also LEDL1.4 (Pin_4), LEDR1.4 (Pin_4)
- net LEDR: now also LEDL1.3 (Pin_3), LEDR1.3 (Pin_3)
- net LEDG: now reaches LEDL1.2 (Pin_2)
- net LEDG: now also LEDR1.2 (Pin_2)
- new net Bat: Lion_Charger1.3 (Pin_3)
- new net EN: Lion_Charger1.4 (Pin_4), SW3.1 (A)
- new net LB: Lion_Charger1.6 (Pin_6)
- new net USB: Lion_Charger1.1 (Pin_1)
- no-connect marks 1 -> 4
