File: 2024-25/Onboarding/jenninbl/led_board/led_board.kicad_sch (KiCad schematic)
At the start: 6 parts, among them J1 Conn_01x08, J2 Conn_01x04, J3 Conn_01x04, SW1 SW_SPST, SW2 SW_SPST, SW3 SW_SPST

Commit message: bruh
Parts:
- SW1, SW2, SW3: footprint (none) -> RB141C1100:SW_RB141C1100
Changed lines of the file:
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@@
 			)
 		)
-		(property "Footprint" ""
+		(property "Footprint" "RB141C1100:SW_RB141C1100"
 			(at 106.68 82.55 0)
 			(effects
@@
 			)
 		)
-		(property "Footprint" ""
+		(property "Footprint" "RB141C1100:SW_RB141C1100"
 			(at 106.68 73.66 0)
 			(effects
@@
 			)
 		)
-		(property "Footprint" ""
+		(property "Footprint" "RB141C1100:SW_RB141C1100"
 			(at 106.68 91.44 0)
 			(effects

Commit message: sus
Connections:
- net GND: now also SW1.2 (B)
- net LEDB: now also SW3.2 (B)
- net LEDR: now also SW2.2 (B)
Changed lines of the file:
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@@
+	(wire
+		(pts
+			(xy 114.3 82.55) (xy 111.76 82.55)
+		)
+		(stroke
+			(width 0)
+			(type default)
+		)
+	)
 	(wire
 		(pts
@@
 	(wire
 		(pts
+			(xy 114.3 91.44) (xy 111.76 91.44)
+		)
+		(stroke
+			(width 0)
+			(type default)
+		)
+	)
+	(wire
+		(pts
+			(xy 114.3 73.66) (xy 111.76 73.66)
+		)
+		(stroke
+			(width 0)
+			(type default)
+		)
+	)
+	(wire
+		(pts
 			(xy 127 91.44) (xy 132.08 91.44)
 		)
@@
 	(label "GND"
 		(at 77.47 76.2 0)
+		(fields_autoplaced yes)
+		(effects
+			(font
+				(size 1.27 1.27)
+			)
+			(justify left bottom)
+		)
+	)
+	(label "LEDR"
+		(at 114.3 82.55 0)
 		(fields_autoplaced yes)
 		(effects
@@
 		)
 	)
+	(label "GND"
+		(at 114.3 73.66 0)
+		(fields_autoplaced yes)
+		(effects
+			(font
+				(size 1.27 1.27)
+			)
+			(justify left bottom)
+		)
+	)
 	(label "LEDB"
 		(at 127 96.52 0)
@@
 		(fields_autoplaced yes)
 		(effects
+			(font
+				(size 1.27 1.27)
+			)
+			(justify left bottom)
+		)
+	)
+	(label "LEDB"
+		(at 114.3 91.44 0)
+		(fields_autoplaced yes)
+		(effects
