File: 2025-26/Armor Panel/Starter/Armor Panel/Armor Panel.kicad_pcb (KiCad board)
At the start: 2 copper layers, 75 x 75 mm, 4 parts

Commit message: My Armor Panel
Parts:
- added CHARGER1: Conn_01x08, Component Library:Power Boost Board, B.Cu at (144.6, 96.8)
- added D2: LB_LED, LED_THT:LED_D5.0mm, B.Cu at (154.0, 112.0)
- added H1: MountingHole_Pad_MP, Component Library:Wire THT Pad, B.Cu at (158.5, 68.0)
- added H2: MountingHole_Pad_MP, Component Library:Wire THT Pad, B.Cu at (164.5, 68.0)
- added H3: MountingHole_Pad_MP, Component Library:Wire THT Pad, B.Cu at (121.5, 68.0)
- added H4: MountingHole_Pad_MP, Component Library:Wire THT Pad, B.Cu at (127.5, 68.0)
- added H5: MountingHole_Pad_MP, Component Library:Wire THT Pad, B.Cu at (144.5, 82.5)
- added H6: MountingHole_Pad_MP, Component Library:Wire THT Pad, B.Cu at (144.5, 76.5)
- added SW1: SW_SPDT_MSM, Component Library:SPDT, B.Cu at (129.0, 57.0)
- added SW_EN1: SW_SPST, Component Library:SPST, B.Cu at (137.5, 65.5)
Routing:
- net /GND: track 0.00 -> 99.5 mm
- net /EN: track 0.00 -> 60.3 mm
- net /5V: track 0.00 -> 32.6 mm
- net /LEDR: track 0.00 -> 23.1 mm
- net /LEDB: track 0.00 -> 17.6 mm

Commit message: Fixed Stuff
Parts:
- added R2: 220, Resistor_THT:R_Axial_DIN0309_L9.0mm_D3.2mm_P12.70mm_Horizontal, F.Cu at (164.8, 102.5)
- moved H1 48.5 mm to (110.0, 69.0)
- moved H3 47.0 mm to (168.0, 74.5)
- moved H6 39.5 mm to (105.5, 82.5)
- moved H5 25.0 mm to (169.5, 82.5)
- moved H4 21.5 mm to (107.0, 74.5)
- moved SW1 3.00 mm to (129.0, 60.0)
- moved H2 1.12 mm to (165.0, 69.0)
- moved SW_EN1 0.50 mm to (137.5, 66.0)
Routing:
- net /5V: track 32.6 -> 179.2 mm
- net /LEDB: track 17.6 -> 113.5 mm
- net /LEDR: track 23.1 -> 69.3 mm
- net /GND: track 99.5 -> 83.9 mm
- net Net-(D2-A): track 0.00 -> 13.0 mm
- net /LB: track 0.00 -> 7.82 mm
- net /EN: track 60.3 -> 63.4 mm

Commit message: Finished board design
Parts:
- CHARGER1: moved to F.Cu
- moved D2 41.4 mm to (137.5, 74.0), turned to -90 degrees
- moved R2 32.9 mm to (144.7, 76.5), turned to 0 degrees
- moved CHARGER1 23.9 mm to (167.2, 88.9), turned to -90 degrees
Routing:
- net /5V: track 179.2 -> 81.7 mm
- net /EN: track 63.4 -> 29.8 mm
- net /GND: track 83.9 -> 69.5 mm
- net /LB: track 7.82 -> 15.9 mm
- net /LEDB: track 113.5 -> 121.3 mm
- net /LEDR: track 69.3 -> 75.8 mm
- net Net-(D2-A): track 13.0 -> 7.15 mm
Other:
- board text added: "5V"
- board text added: "EN"
- board text added: "GND"
- board text added: "LEDB"
- board text added: "LEDR"

Commit message: Unholy Abomination
Parts:
- removed H1, H2, H3, H4, H5, H6: MountingHole_Pad_MP, Component Library:Wire THT Pad
- removed SW1: SW_SPDT_MSM, Component Library:SPDT
- removed SW_EN1: SW_SPST, Component Library:SPST
- added J1: Conn_01x03, Connector_JST:JST_PH_B3B-PH-K_1x03_P2.00mm_Vertical, F.Cu at (107.5, 80.5)
- added J2: Conn_01x03, Connector_JST:JST_PH_B3B-PH-K_1x03_P2.00mm_Vertical, F.Cu at (167.0, 80.5)
- added J3: Conn_01x03, Connector_JST:JST_PH_B3B-PH-K_1x03_P2.00mm_Vertical, F.Cu at (125.5, 61.0)
- added J4: Conn_01x02, Connector_JST:JST_PH_B2B-PH-K_1x02_P2.00mm_Vertical, F.Cu at (146.0, 116.0)
- added J5: Conn_01x02, Connector_JST:JST_PH_B2B-PH-K_1x02_P2.00mm_Vertical, F.Cu at (151.5, 65.0)
- D2: moved to F.Cu
- moved D2 11.1 mm to (139.0, 63.0)
- moved R2 2.12 mm to (146.2, 78.0)
- moved CHARGER1 0.43 mm to (167.2, 88.5)
Routing:
- net /5V: track 81.7 -> 142.3 mm
- net /GND: track 69.5 -> 109.0 mm
- net /USB: track 0.00 -> 28.9 mm
- net /LEDB: track 121.3 -> 96.1 mm
- net Net-(D2-A): track 7.15 -> 17.6 mm
- net /LEDR: track 75.8 -> 83.8 mm
- net /LB: track 15.9 -> 11.8 mm
- net /EN: track 29.8 -> 25.8 mm
Other:
- board text removed: "5V"
- board text removed: "EN"
- board text removed: "GND"
- board text removed: "LEDB"
- board text removed: "LEDR"
