File: 2025-26/Measurement Testing/Measurement Testing/Measurement Testing.kicad_sch (KiCad schematic)
At the start: 5 parts, among them J1 Power Supply, U2 INA240A2PWR

Commit message: Still working
Parts:
- added J2: XT30PW-F, XT30PW-F:AMASS_XT30PW-F, symbol XT30PW-F:XT30PW-F
Connections:
- net GND: now also J2.N
- net at R1.1, Rshunt.2, U2.3: now also J2.P

Commit message: Finished basic schematic
Parts:
- added C1, C4, C5: 1 uF, symbol Device:C
- added C2: 22 uF, symbol Device:C
- added C3, C6: 10 uF, symbol Device:C
- added R3: 100k, symbol Device:R
- added U3: RASPBERRY_PI_PICO, RASPBERRY_PI_PICO:RASPBERRY_PI_PICO, symbol RASPBERRY_PI_PICO:RASPBERRY_PI_PICO
- added U4: ADS8684IDBTR, ADS8684IDBTR:SOP50P640X120-38N, symbol ADS8684IDBTR:ADS8684IDBTR
- R1: value R -> 8.2k
- R2: value R -> 1k
- Rshunt: value R -> 5m
Connections:
- net GND: now also U2.1, U2.4, U2.6, U2.7, C1.2, C2.2, C3.2, C4.2, C5.2, C6.2, U4.10 (AUX_IN), U4.11 (AUX_GND), U4.12 (NC), U4.13 (NC__1), U4.14 (NC__2), U4.15 (NC__3), U4.17 (AIN_0GND), U4.19 (AIN_1GND), U4.20 (AIN_2GND), U4.21 (AIN_2P), U4.22 (AIN_3GND), U4.23 (AIN_3P), U4.24 (NC__4), U4.25 (NC__5), U4.26 (NC__6), U4.27 (NC__7), U4.28 (AGND__1), U4.29 (AGND__2), U4.3 (DAISY), U4.31 (AGND__3), U4.32 (AGND__4), U4.33 (DGND), U4.4 (~{REFSEL}), U4.6 (REFGND), U4.8 (AGND)
- net at R1.2, R2.1: now also U4.18 (AIN_1P)
- net at U2.8: now also U4.16 (AIN_0P)
- new net: U3.GP19, U4.1 (SDI)
- new net: C5.1, U4.30 (AVDD__1)
- new net: C6.1, U4.34 (DVDD)
- new net: U3.GP16, U4.36 (SDO)
- new net: U3.GP18, U4.37 (SCLK)
- new net: U3.GP17, U4.38 (~{CS})
- new net: C3.1, U4.5 (REFIO)
- new net: C1.1, C2.1, U4.7 (REFCAP)
- new net: C4.1, U4.9 (AVDD)
- new net: R3.2, U3.3V3_EN
- new net: R3.1, U3.VBUS, U3.VSYS
Other:
- moved on the sheet: J2, R1, R2

Commit message: Some board thingy
Parts:
- C1, C4, C5: footprint (none) -> Measurement:CAPC1608X90N
- C2: footprint (none) -> Measurement:CAPC3225X270N
- C3, C6: footprint (none) -> Measurement:CAPC2012X140N
- J1: footprint (none) -> Connector_PinHeader_1.00mm:PinHeader_1x02_P1.00mm_Vertical
- R1: footprint (none) -> Measurement:CAPC1005X55N
- R2, R3: footprint (none) -> Measurement:RESC1607X60N
- Rshunt1: renamed from Rshunt; footprint (none) -> Measurement:RESC6331X55N
