File: 2025-26/Control Board/Control Board V3/5vpsu.kicad_sch (KiCad schematic)
At the start: 0 parts

Commit message: board almost fully designed
i want to try a different orientation so gonna push this so i can easily revert
Parts:
- added C17: 100 nF, Capacitor_SMD:C_0402_1005Metric, symbol Device:C
- added C18: 47u, Capacitor_SMD:C_0805_2012Metric, symbol Device:C
- added C19: 10u, Capacitor_SMD:C_1206_3216Metric, symbol Device:C
- added D4: D_Zener, Diode_SMD:D_SOD-323F, symbol Device:D_Zener
- added L1: 13u, Inductor_SMD:L_Wuerth_WE-PDF, symbol Device:L
- added R8: 10k, Resistor_SMD:R_0603_1608Metric, symbol Device:R
- added Rfbb1: 13.7k, Resistor_SMD:R_0402_1005Metric_Pad0.72x0.64mm_HandSolder, symbol Device:R
- added Rfbt1: 100k, Resistor_SMD:R_0402_1005Metric_Pad0.72x0.64mm_HandSolder, symbol Device:R
- added U5: TPS54308DDCR, Package_TO_SOT_SMD:SOT-23-6, symbol TPS54308DDCR:TPS54308DDCR
Connections:
- new net: C17.1, U5.6 (BOOT)
- new net: C17.2, L1.1, U5.2 (SW)
- new net: Rfbb1.1, Rfbt1.2, U5.4 (FB)
- new net: D4.1 (K), R8.1, U5.5 (EN)
- new net 5V: C18.1, L1.2, Rfbt1.1
- new net D_GND: C18.2, Rfbb1.2
- new net PSU_GND: C19.2, D4.2 (A), U5.1 (GND)
- new net PSU_Vin: C19.1, R8.2, U5.3 (VIN)
