File: 2025-26/Control Board/Control Board V3/measurements2.kicad_sch (KiCad schematic)
At the start: 0 parts

Commit message: board almost fully designed
i want to try a different orientation so gonna push this so i can easily revert
Parts:
- added C13: 22 uF, Capacitor_SMD:C_1210_3225Metric, symbol Device:C
- added C14, C15, C3: 1 uF, Capacitor_SMD:C_0603_1608Metric, symbol Device:C
- added C16, C4: 10 uF, Capacitor_SMD:C_0805_2012Metric, symbol Device:C
- added C21, C28: 100 nF, Capacitor_SMD:C_0402_1005Metric, symbol Device:C
- added R3: 8.2k, Resistor_SMD:R_0603_1608Metric, symbol Device:R
- added R4: 1k, Resistor_SMD:R_0603_1608Metric, symbol Device:R
- added Rshunt2: 5m, Resistor_SMD:R_2512_6332Metric, symbol Device:R
- added U1: ADS8684IDBTR, Package_SO:TSSOP-38_4.4x9.7mm_P0.5mm, symbol ADS8684IDBTR:ADS8684IDBTR
- added U2, U6: INA240A2PWR, Package_SO:TSSOP-8_4.4x3mm_P0.65mm, symbol INA240A2PWR:INA240A2PWR
Connections:
- new net: U1.16 (AIN_0P), U2.8
- new net: C13.1, C15.1, U1.7 (REFCAP)
- new net: U1.21 (AIN_2P), U6.8
- new net: C16.1, U1.5 (REFIO)
- new net: R3.1, R4.1, U1.18 (AIN_1P)
- new net 3V3: C4.1, U1.2 (~{RST}/~{PD}), U1.34 (DVDD)
- new net 5V: C14.1, C21.2, C28.1, C3.1, U1.30 (AVDD__1), U1.9 (AVDD), U2.5, U6.5
- new net CM01: R3.2, Rshunt2.2, U2.3, U6.2
- new net DGND: C21.1, C28.2, C4.2, R4.2, U1.3 (DAISY), U1.33 (DGND), U1.4 (~{REFSEL}), U2.1, U2.4, U2.6, U2.7, U6.1, U6.4, U6.6, U6.7
- new net PGND: C13.2, C14.2, C15.2, C16.2, C3.2, U1.10 (AUX_IN), U1.11 (AUX_GND), U1.12 (NC), U1.13 (NC__1), U1.14 (NC__2), U1.15 (NC__3), U1.17 (AIN_0GND), U1.19 (AIN_1GND), U1.20 (AIN_2GND), U1.22 (AIN_3GND), U1.23 (AIN_3P), U1.24 (NC__4), U1.25 (NC__5), U1.26 (NC__6), U1.27 (NC__7), U1.28 (AGND__1), U1.29 (AGND__2), U1.31 (AGND__3), U1.32 (AGND__4), U1.6 (REFGND), U1.8 (AGND)
- new net SPI1_CLK: U1.37 (SCLK)
- new net SPI1_CS: U1.38 (~{CS})
- new net SPI1_MISO: U1.36 (SDO)
- new net SPI1_MOSI: U1.1 (SDI)
- new net V_cap: Rshunt2.1, U2.2, U6.3
