File: 2025-26/Control Board/Control Board V3/Control Board V3.kicad_sch (KiCad schematic)
At the start: 23 parts, among them J1 PM01, J10 J_5V, J11 UART, J2 CM01, J3 Mini PC, J4 Motor 1, J5 Motor 2, J6 Motor 3, J7 Motor 4, J8 Motor 0, J9 J_GND, SW1 SW_DPDT_x2

Commit message: so much..
so, not much change to pcbs, mainly the job files are now included.

on the controls side there is a vibe coded mess that needs to be cleaned up. making a checkpoint because i want to see if a separate claude chat can clean up the code first.
Parts:
- added J12: Motor 1, Connector_AMASS:AMASS_XT30PW-M_1x02_P2.50mm_Horizontal, symbol Connector:Conn_01x02_Pin
- added J13: Motor 2, Connector_AMASS:AMASS_XT30PW-M_1x02_P2.50mm_Horizontal, symbol Connector:Conn_01x02_Pin
- added J14: Motor 3, Connector_AMASS:AMASS_XT30PW-M_1x02_P2.50mm_Horizontal, symbol Connector:Conn_01x02_Pin
- added J15: Motor 4, Connector_AMASS:AMASS_XT30PW-M_1x02_P2.50mm_Horizontal, symbol Connector:Conn_01x02_Pin
- added J16: Motor 0, Connector_AMASS:AMASS_XT30PW-M_1x02_P2.50mm_Horizontal, symbol Connector:Conn_01x02_Pin
- added J17: PM01, Connector_AMASS:AMASS_XT30PW-M_1x02_P2.50mm_Horizontal, symbol Connector:Conn_01x02_Pin
- H1, H2, H3, H4: now in the parts list
- J1, J10, J11, J2, J3, J4, J5, J6, J7, J8, J9: now left out of the parts list
Connections:
- net DGND: now also A1.13 (GND), A1.18 (GND), A1.23 (GND), A1.28 (GND), A1.3 (GND), A1.33 (AGND), A1.38 (GND), A1.8 (GND)
- net PGND: now also J12.1 (Pin_1), J13.1 (Pin_1), J14.1 (Pin_1), J15.1 (Pin_1), J16.1 (Pin_1), J17.1 (Pin_1)
- net PM01: now also J17.2 (Pin_2)
- net PWM_H: now also A1.19 (GPIO14); no longer A1.20 (GPIO15)
- net PWM_L: now also A1.20 (GPIO15); no longer A1.19 (GPIO14)
- net V_DT: now also J12.2 (Pin_2), J13.2 (Pin_2), J14.2 (Pin_2), J15.2 (Pin_2), J16.2 (Pin_2)
- net at J11.1 (Pin_1): now also A1.2 (GPIO1); no longer A1.12 (GPIO9)
- net at J11.2 (Pin_2): now also A1.1 (GPIO0); no longer A1.11 (GPIO8)
Other:
- sheet Measurement System 1 ports: added PGND; removed none
- sheet Measurement System 2 ports: added PGND; removed none
- moved on the sheet: J11
