File: 2026-27/Control Board/Control Board V3/measurements1.kicad_sch (KiCad schematic)
At the start: 12 parts, among them U3 ADS8684IDBTR, U4 INA240A2PWR

Commit message: push
Parts:
- removed C10, C11: 1 uF, Capacitor_SMD:C_0603_1608Metric, symbol Device:C
- removed C12, C2: 10 uF, Capacitor_SMD:C_0805_2012Metric, symbol Device:C
- removed C20: 100 nF, Capacitor_SMD:C_0402_1005Metric, symbol Device:C
- removed C9: 22 uF, Capacitor_SMD:C_1210_3225Metric, symbol Device:C
- added R10: 10k, symbol Device:R
- added R9: 90k, symbol Device:R
- C1: value 1 uF -> C; footprint Capacitor_SMD:C_0603_1608Metric -> (none)
- R1: value 8.2k -> 10k; footprint Resistor_SMD:R_0603_1608Metric -> (none)
- R2: value 1k -> 16k; footprint Resistor_SMD:R_0603_1608Metric -> (none)
Connections:
- net 3V3: no longer U3.34 (DVDD)
- net DGND: no longer U3.33 (DGND)
- net PM01: now also R9.1; no longer R1.1
- net at U3.16 (AIN_0P), U4.8: no longer U3.21 (AIN_2P)
- net GND: now reaches R1.2, R2.1
- net GND: now also C1.2, R2.2, U3.17 (AIN_0GND), U3.19 (AIN_1GND), U4.1, U4.4, U4.6, R10.2; no longer U3.18 (AIN_1P)
- net at U3.5 (REFIO): now also R1.1
- net 5V renamed +5V
- net +5V: no longer U3.30 (AVDD__1), U3.9 (AVDD)
- removed net PGND: C1.2, R2.2, U3.10 (AUX_IN), U3.11 (AUX_GND), U3.12 (NC), U3.13 (NC__1), U3.14 (NC__2), U3.15 (NC__3), U3.17 (AIN_0GND), U3.19 (AIN_1GND), U3.20 (AIN_2GND), U3.22 (AIN_3GND), U3.23 (AIN_3P), U3.24 (NC__4), U3.25 (NC__5), U3.26 (NC__6), U3.27 (NC__7), U3.28 (AGND__1), U3.29 (AGND__2), U3.31 (AGND__3), U3.32 (AGND__4), U3.6 (REFGND), U3.8 (AGND), U4.1, U4.4, U4.6, U4.7
- new net: R10.1, R9.2, U3.18 (AIN_1P)
